File: hardware/Steve 68k.kicad_sch (KiCad schematic)
At the start: 52 parts, among them IC1 MC68008FN8, J1 Conn_02x32_Odd_Even, J2 Serial 1, J3 Serial 2, J4 CLK Select, J5 I2C, SW1 Reset, U1 74LS32, U10 74HC04, U2 28C256, U3 GAL16V8, U4 74HC04, U5 MC68681FN, U6 74HC04, U7 AS6C4008-55PCN, U8 Max705, U9 PCA9564, X1 CXO_DIP8, X2 1.8432 Mhz

Commit message: Rev V20220601
Parts:
- removed C13, C5: .1uF, Capacitor_SMD:C_0603_1608Metric, symbol Device:C
- removed R14: 10k, symbol Device:R
- removed U10, U6: 74HC04, symbol 74xx:74HC04
- removed U9: PCA9564, symbol mc68k:PCA9564
Connections:
- net 68681_Int: no longer IC1.46 (~{IPL2}), J1.52 (Pin_52), R2.2
- new net ~{IPL2}: IC1.46 (~{IPL2}), J1.52 (Pin_52), R2.2
- no-connect marks 23 -> 18

Commit message: Latest version sent for fab
Parts:
- removed J2: Serial 1, Connector_PinHeader_2.54mm:PinHeader_1x04_P2.54mm_Vertical, symbol Connector:Conn_01x04_Male
- removed J3: Serial 2, Connector_PinHeader_2.54mm:PinHeader_1x04_P2.54mm_Vertical, symbol Connector:Conn_01x04_Male
- removed J5: I2C, symbol Connector:Conn_01x04_Male
- removed X2: 1.8432 Mhz, Oscillator:Oscillator_DIP-14, symbol Oscillator:CXO_DIP14
- added C13: 100uF, Capacitor_SMD:CP_Elec_4x5.4, symbol Device:C_Polarized
- added C5: 12pf, Capacitor_SMD:C_0603_1608Metric, symbol Device:C
- added D6: PWR, LED_SMD:LED_1206_3216Metric, symbol Device:LED
- added D7: ERR, LED_SMD:LED_1206_3216Metric, symbol Device:LED
- added J2: 5V Input, Connector_BarrelJack:BarrelJack_Horizontal, symbol Connector:Barrel_Jack
- added J3: Serial 1, Connector_PinSocket_2.54mm:PinSocket_1x06_P2.54mm_Vertical, symbol Connector:Conn_01x06_Female
- added J6: Serial 2, Connector_PinSocket_2.54mm:PinSocket_1x06_P2.54mm_Vertical, symbol Connector:Conn_01x06_Female
- added R14, R15, R16: 10k, Resistor_SMD:R_0603_1608Metric, symbol Device:R
- added R17, R18: 220, Resistor_SMD:R_0603_1608Metric, symbol Device:R
- added U6: L7805, Package_TO_SOT_THT:TO-220-3_Horizontal_TabUp, symbol Regulator_Linear:L7805
- added Y1: 3.6864, Crystal:Crystal_HC49-U_Vertical, symbol Device:Crystal
- C9: value .1uF -> 12pf
- U4: footprint Package_SO:SOIC-14_3.9x8.7mm_P1.27mm -> Package_SO:SOIC-14W_7.5x9mm_P1.27mm
- U8: footprint Package_DIP:DIP-8_W7.62mm_Socket_LongPads -> Package_SO:SOIC-8_3.9x4.9mm_P1.27mm
Connections:
- net A17: now also U3.11 (I10/~{OE})
- net A18: now also U3.1 (I1/CLK)
- net CLK: no longer U3.1 (I1/CLK)
- net GND: now also C9.1, C5.1, D7.1 (K), J3.6 (Pin_6), J6.6 (Pin_6); no longer C9.2, U3.11 (I10/~{OE})
- net RxDA: now also J3.3 (Pin_3)
- net RxDB: now also J6.3 (Pin_3)
- net TxDA: now also J3.2 (Pin_2)
- net TxDB: now also J6.2 (Pin_2)
- net VCC: now also C13.1, J3.4 (Pin_4), J6.4 (Pin_4), R14.1, R15.1, R16.1, R17.1, U6.3 (OUT); no longer C9.1
- net ~{DTACK_UART}: now also R14.2
- net ~{DTACK_USER}: now also R16.2
- net ERROR: now reaches U3.17 (I03)
- net ERROR: now also R18.1
- net 68681_X2: now reaches U5.37 (X2)
- net 68681_X2: now also C9.2, Y1.1
- net DTACK_I2C renamed ~{DTACK_I2C}
- net ~{DTACK_I2C}: now also R15.2
- net IP0 renamed CTSA
- net CTSA: now also J3.5 (Pin_5)
- net IP1 renamed CTSB
- net CTSB: now also J6.5 (Pin_5)
- net OP0 renamed RTSA
- net OP2 renamed RTSB
- net UART_CLK renamed 68681_X1
- net 68681_X1: now also C5.2, Y1.2
- new net: C13.2, D6.1 (K), J2.2, U6.2 (GND)
- new net: D7.2 (A), R18.2
- new net: J2.1, U6.1 (IN)
- new net: D6.2 (A), R17.2
- new net DTRA: J3.1 (Pin_1)
- new net DTRB: J6.1 (Pin_1)
- no-connect marks 18 -> 15
Other:
- note added: "5VDC"
- note added: "CPU CLK"
- note added: "Power"
- note added: "UART CLK"
- note removed: "RX"
- note removed: "TX"
- moved on the sheet: C10, C11, C3, D1, D2, D3, D4, D5, J4, R5, R6, R7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

Commit message: V20220905 sent for fab
Parts:
- removed C1, C8: .1uF, Capacitor_SMD:C_0603_1608Metric, symbol Device:C
- removed C13: 100uF, Capacitor_SMD:CP_Elec_4x5.4, symbol Device:C_Polarized
- removed C15: 10uF, Capacitor_SMD:CP_Elec_4x5.4, symbol Device:C_Polarized
- removed C5, C9: 12pf, Capacitor_SMD:C_0603_1608Metric, symbol Device:C
- removed D3: RAM, LED_SMD:LED_1206_3216Metric, symbol Device:LED
- removed D4: UART, LED_SMD:LED_1206_3216Metric, symbol Device:LED
- removed D5: USER, LED_SMD:LED_1206_3216Metric, symbol Device:LED
- removed D6: PWR, LED_SMD:LED_1206_3216Metric, symbol Device:LED
- removed D7: ERR, LED_SMD:LED_1206_3216Metric, symbol Device:LED
- removed J1: Conn_02x32_Odd_Even, Connector_PinHeader_2.54mm:PinHeader_2x32_P2.54mm_Vertical, symbol Connector_Generic:Conn_02x32_Odd_Even
- removed J2: 5V Input, Connector_BarrelJack:BarrelJack_Horizontal, symbol Connector:Barrel_Jack
- removed J4: CLK Select, Connector_PinHeader_2.54mm:PinHeader_1x03_P2.54mm_Vertical, symbol Connector:Conn_01x03_Male
- removed J6: Serial 2, Connector_PinSocket_2.54mm:PinSocket_1x06_P2.54mm_Vertical, symbol Connector:Conn_01x06_Female
- removed R14, R15, R16: 10k, Resistor_SMD:R_0603_1608Metric, symbol Device:R
- removed R17, R18: 220, Resistor_SMD:R_0603_1608Metric, symbol Device:R
- removed U3: GAL16V8, Package_DIP:DIP-20_W7.62mm_Socket_LongPads, symbol Logic_Programmable:GAL16V8
- removed unit 6 of U4
- removed unit 3 of U4
- removed unit 4 of U4
- removed unit 5 of U4
- removed unit 2 of U4
- removed U5: MC68681FN, Package_LCC:PLCC-44_THT-Socket, symbol mc68k:MC68681FN
- removed U6: L7805, Package_TO_SOT_THT:TO-220-3_Horizontal_TabUp, symbol Regulator_Linear:L7805
- removed Y1: 3.6864, Crystal:Crystal_HC49-U_Vertical, symbol Device:Crystal
- added C11: 100uF, Capacitor_SMD:CP_Elec_4x5.4, symbol Device:C_Polarized
- added C12, C3, C6: .1uF, Capacitor_SMD:C_0603_1608Metric, symbol Device:C
- added J1: Power, Connector_PinHeader_2.54mm:PinHeader_1x03_P2.54mm_Vertical, symbol Connector:Conn_01x03_Male
- added J2: I2C, Connector_PinSocket_2.54mm:PinSocket_1x04_P2.54mm_Vertical, symbol Connector:Conn_01x04_Male
- added J3: Debug, Connector_PinHeader_2.54mm:PinHeader_2x34_P2.54mm_Vertical, symbol Connector_Generic:Conn_02x34_Odd_Even
- added J4: ICSP, Connector_PinSocket_2.54mm:PinSocket_2x03_P2.54mm_Vertical, symbol Connector_Generic:Conn_02x03_Counter_Clockwise
- added unit 6 of U1
- added unit 5 of U1
- added unit 3 of U1
- added unit 4 of U1
- added unit 2 of U1
- added U3: 74HC138, Package_SO:SOIC-16_3.9x9.9mm_P1.27mm, symbol 74xx:74LS138
- added U4: 74HC257, Package_SO:SOIC-16_3.9x9.9mm_P1.27mm, symbol 74xx:74LS257
- added U7: ATmega1284P-P, Package_DIP:DIP-40_W15.24mm, symbol MCU_Microchip_ATmega:ATmega1284P-P
- D1: value I2C -> PWR LED
- D2: value ROM -> BLINK LED
- R12, R13: value 10k -> 220
- R5, R6, R7, R8, R9: value 220 -> 10k
- U1: renamed from U4; footprint Package_SO:SOIC-14W_7.5x9mm_P1.27mm -> Package_SO:SOIC-14_3.9x8.7mm_P1.27mm
- U2: renamed from U1; value 74LS32 -> 74HC32
- X1: value CXO_DIP8 -> 8Mhz
- renumbered C12 to C1, C11 to C10, C3 to C4, C4 to C5, C6 to C7, C7 to C8, C10 to C9, J3 to J5, U7 to U5, U2 to U6
Connections:
- net CLK_ONBOARD is gone; now on net CLK: X1.5 (OUT)
- net A0: now also J3.3 (Pin_3), U7.1 (PB0)
- net A1: now also J3.4 (Pin_4), U7.2 (PB1)
- net A10: now also J3.13 (Pin_13)
- net A11: now also J3.14 (Pin_14)
- net A12: now also J3.15 (Pin_15)
- net A13: now also J3.16 (Pin_16)
- net A14: now also J3.17 (Pin_17)
- net A15: now also J3.18 (Pin_18)
- net A16: now also J3.19 (Pin_19)
- net A17: now also J3.20 (Pin_20)
- net A18: now also J3.21 (Pin_21)
- net A19: now also J3.22 (Pin_22), U3.1 (A0)
- net A2: now also J3.5 (Pin_5), U7.3 (PB2)
- net A20: now also J3.23 (Pin_23), U3.2 (A1)
- net A21: now also J3.24 (Pin_24), U3.3 (A2)
- net A3: now also J3.6 (Pin_6), U7.4 (PB3)
- net A4: now also J3.7 (Pin_7), U7.5 (PB4)
- net A5: now also J3.8 (Pin_8), U7.24 (PC2)
- net A6: now also J3.9 (Pin_9), U7.25 (PC3)
- net A7: now also J3.10 (Pin_10), U7.26 (PC4)
- net A8: now also J3.11 (Pin_11), U7.27 (PC5)
- net A9: now also J3.12 (Pin_12), U7.17 (PD3)
- net CLK: now also J3.42 (Pin_42), U7.13 (XTAL1)
- net D0: now also J3.27 (Pin_27), U7.40 (PA0)
- net D1: now also J3.28 (Pin_28), U7.39 (PA1)
- net D2: now also J3.29 (Pin_29), U7.38 (PA2)
- net D3: now also J3.30 (Pin_30), U7.37 (PA3)
- net D4: now also J3.31 (Pin_31), U7.36 (PA4)
- net D5: now also J3.32 (Pin_32), U7.35 (PA5)
- net D6: now also J3.33 (Pin_33), U7.34 (PA6)
- net D7: now also J3.34 (Pin_34), U7.33 (PA7)
- net E: now also J3.51 (Pin_51)
- net FC0: now also J3.60 (Pin_60)
- net FC1: now also J3.61 (Pin_61)
- net FC2: now also J3.62 (Pin_62)
- net GND: now also R12.1, R13.1, C11.2, C12.2, C3.2, C6.2, J1.3 (Pin_3), J2.2 (Pin_2), J3.1 (Pin_1), J3.2 (Pin_2), J4.4 (Pin_4), U1.11, U1.13, U1.3, U1.5, U1.9, U3.4 (E1), U3.5 (E2), U3.8 (GND), U4.10 (I1d), U4.11 (I0d), U4.13 (I1c), U4.14 (I0c), U4.15 (OE), U4.5 (I0b), U4.6 (I1b), U4.8 (GND), U7.11 (GND), U7.31 (GND); no longer D1.1 (K), D2.1 (K)
- net R~{W}: now also J3.43 (Pin_43), U7.16 (PD2)
- net VCC: now also D1.2 (A), R5.1, R6.1, R7.1, R8.1, R9.1, C11.1, C12.1, C3.1, C6.1, J1.1 (Pin_1), J2.1 (Pin_1), J3.67 (Pin_67), J3.68 (Pin_68), J4.6 (Pin_6), U3.16 (VCC), U3.6 (E3), U4.16 (VCC), U7.10 (VCC), U7.30 (AVCC); no longer R12.1, R13.1
- net ~{AS}: now also R10.2, J3.44 (Pin_44), U4.3 (I1a)
- net ~{BERR}: now also R4.2, J3.49 (Pin_49); no longer R11.2
- net ~{BGACK}: now also R8.2, J3.53 (Pin_53); no longer R13.2
- net ~{BG}: now also J3.56 (Pin_56)
- net ~{BR}: now also R7.2, J3.55 (Pin_55); no longer R12.2
- net ~{DS}: now also J3.46 (Pin_46)
- net ~{DTACK_CPU}: now also R11.2, J3.50 (Pin_50), U4.4 (Za)
- net ~{HALT}: now also R6.2, J3.48 (Pin_48); no longer R10.2
- net ~{IPL0}: now also J3.57 (Pin_57)
- net ~{IPL1}: now also J3.58 (Pin_58)
- net ~{IPL2}: now also J3.59 (Pin_59)
- net ~{RAMSEL}: now also J3.64 (Pin_64), U3.14 (O1)
- net ~{RESET}: now also J3.47 (Pin_47), J4.3 (Pin_3), U7.9 (~{RESET})
- net ~{ROMSEL}: now also J3.63 (Pin_63), U3.15 (O0)
- net at D2.2 (A): now also U7.18 (PD4); no longer R7.2
- net ~{DTACK_AVR}: now reaches R9.2
- net ~{DTACK_AVR}: now also U4.2 (I0a), U7.28 (PC6)
- net ~{VPA}: now reaches R5.2
- net ~{VPA}: now also IC1.43 (~{VPA}), J3.54 (Pin_54); no longer D1.2 (A)
- removed net 68681_Int: IC1.43 (~{VPA}), R4.2
- net CTSA: no longer names the net of J5.5 (Pin_5)
- net DTRA: no longer names the net of J5.1 (Pin_1)
- net RxDA renamed RXD0
- net RXD0: now also U7.14 (PD0)
- net TxDA renamed TXD0
- net TXD0: now also U7.15 (PD1)
- new net: D2.1 (K), R13.2
- new net: D1.1 (K), R12.2
- new net IPL0: U7.19 (PD5)
- new net IPL1: U7.20 (PD6)
- new net IPL2: U7.21 (PD7)
- new net MISO: J4.1 (Pin_1), U7.7 (PB6)
- new net MOSI: J4.5 (Pin_5), U7.6 (PB5)
- new net SCK: J4.2 (Pin_2), U7.8 (PB7)
- new net SCL: J2.4 (Pin_4), U7.22 (PC0)
- new net SDA: J2.3 (Pin_3), U7.23 (PC1)
- new net ~{AVRSEL}: J3.65 (Pin_65), U3.13 (O2), U4.1 (S), U7.29 (PC7)
- no-connect marks 15 -> 36
Other:
- note added: "0x0000-0x7FFF"
- note added: "0x10000-"
- note added: "0x180000 start address"
- note added: "0x8000-0xFFFF"
- note added: "AVR controls Serial, I2C and SPI as well as other simpler things. It can address 1024 (1k) bytes."
- note added: "Connectors"
- note added: "IF AVRSEL is LOW then DTACK will be DTACK_AVR otherwise it's the AS"
- note added: "This connector has empty spaces so that the same bus can be used with processors that have 16 data lines and other control lines."
- note added: "Will set OE low if RW is HIGH (READ) and DS is LOW"
- note added: "Will set RAM_WE LOW when RW is LOW (WRITE) AND DS is LOW"
- note removed: "5VDC"
- note removed: "Power"
- note removed: "UART CLK"
- moved on the sheet: C1, C10, C2, C4, C5, C7, C8, C9, IC1, SW1, U1A, U1G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

Commit message: Initial Commit
Parts:
- removed C10, C12, C9: .1uF, Capacitor_SMD:C_0603_1608Metric, symbol Device:C
- removed D2: BLINK LED, LED_SMD:LED_1206_3216Metric, symbol Device:LED
- removed J2: I2C, Connector_PinSocket_2.54mm:PinSocket_1x04_P2.54mm_Vertical, symbol Connector:Conn_01x04_Male
- removed J4: ICSP, Connector_PinSocket_2.54mm:PinSocket_2x03_P2.54mm_Vertical, symbol Connector_Generic:Conn_02x03_Counter_Clockwise
- removed J5: Serial 1, Connector_PinSocket_2.54mm:PinSocket_1x06_P2.54mm_Vertical, symbol Connector:Conn_01x06_Female
- removed R1, R2, R3: 10k, Resistor_SMD:R_0603_1608Metric, symbol Device:R
- removed R13: 220, Resistor_SMD:R_0603_1608Metric, symbol Device:R
- removed unit 6 of U1
- removed unit 5 of U1
- removed unit 3 of U1
- removed unit 4 of U1
- removed unit 7 of U1
- removed unit 2 of U1
- removed unit 3 of U2
- removed unit 4 of U2
- removed unit 5 of U2
- removed U7: ATmega1284P-P, Package_DIP:DIP-40_W15.24mm, symbol MCU_Microchip_ATmega:ATmega1284P-P
- added C? (x2): 22pf, symbol Device:C
- added C? (x5): .1uF, Capacitor_SMD:C_0603_1608Metric, symbol Device:C
- added J?: UART_A, rosco_m68k:1X06, symbol Connector:Conn_01x06_Male
- added J?: UART_B, rosco_m68k:1X06, symbol Connector:Conn_01x06_Male
- added J?: Conn_01x06, rosco_m68k:1X06, symbol Connector_Generic:Conn_01x06
- added Q?: 3.6864MHz, Crystal:Crystal_HC49-4H_Vertical, symbol Device:Crystal
- added R? (x4): 10k, Resistor_SMD:R_0603_1608Metric, symbol Device:R
- added U? (x3): ATF22V10C, symbol rosco:ATF22V10C
- added U?: 68681, symbol Interface:68681
- added U?: 68008D, symbol CPU_NXP_68000:68008D
Connections:
- net A0: now also U?.46 (A0), U?.7 (IN)
- net A1: now also U?.1 (RS1), U?.47 (A1), U?.8 (IN)
- net A10: now also U?.8 (A10)
- net A11: now also U?.9 (A11)
- net A12: now also U?.10 (A12)
- net A13: now also U?.11 (A13)
- net A14: now also U?.12 (A14)
- net A15: now also U?.14 (A15)
- net A16: now also U?.16 (A16)
- net A17: now also U?.17 (A17), U?.4 (IN/PD)
- net A18: now also U?.18 (A18), U?.5 (IN)
- net A19: now also U?.19 (A19), U?.6 (IN)
- net A2: now also U?.3 (RS2), U?.48 (A2), U?.9 (IN)
- net A3: now also U?.1 (A3), U?.5 (RS3)
- net A4: now also U?.2 (A4), U?.6 (RS4)
- net A5: now also U?.3 (A5)
- net A6: now also U?.4 (A6)
- net A7: now also U?.5 (A7)
- net A8: now also U?.6 (A8)
- net A9: now also U?.7 (A9)
- net CLK: now also U?.34 (CLK)
- net D0: now also U?.25 (D0), U?.27 (D0)
- net D1: now also U?.16 (D1), U?.26 (D1)
- net D2: now also U?.24 (D2), U?.25 (D2)
- net D3: now also U?.17 (D3), U?.24 (D3)
- net D4: now also U?.23 (D4), U?.23 (D4)
- net D5: now also U?.18 (D5), U?.22 (D5)
- net D6: now also U?.21 (D6), U?.22 (D6)
- net D7: now also U?.19 (D7), U?.20 (D7)
- net E: now also U?.38 (E)
- net FC0: now also U?.4 (IN/PD), U?.45 (FC0)
- net FC1: now also U?.44 (FC1), U?.5 (IN)
- net FC2: now also U?.43 (FC2), U?.6 (IN)
- net GND: now also C?.2, C?.2, C?.2, C?.2, C?.2, C?.2, C?.2, J?.1 (Pin_1), J?.1 (Pin_1), J?.6 (Pin_6), U?.12 (GND), U?.12 (GND), U?.12 (GND), U?.15 (GND), U?.20 (GND), U?.35 (GND)
- net R~{W}: now also U?.3 (IN), U?.30 (R/W), U?.6 (IN), U?.8 (R/W)
- net VCC: now also C?.1, C?.1, C?.1, C?.1, C?.1, J?.3 (Pin_3), J?.3 (Pin_3), J?.5 (Pin_5), R?.1, R?.1, R?.1, R?.1, U?.13 (VCC), U?.24 (VCC), U?.24 (VCC), U?.24 (VCC), U?.40 (VCC)
- net ~{AS}: now also U?.1 (CLK/IN), U?.2 (IN), U?.28 (AS), U?.4 (IN/PD)
- net ~{BG}: now also U?.32 (BG)
- net ~{DS}: now also U?.2 (IN), U?.29 (DS), U?.5 (IN)
- net ~{IPL1}: now also U?.41 (IPL1)
- net ~{OE}: now also U?.23 (I/O)
- net ~{RAMSEL}: now also U?.1 (CLK/IN), U?.23 (I/O)
- net ~{RAM_WE}: now also U?.22 (I/O)
- net ~{RESET}: now also U?.34 (RESET), U?.37 (RESET)
- net ~{ROMSEL}: now also U?.2 (IN), U?.22 (I/O)
- new net: C?.1, Q?.1, U?.33 (X2)
- new net: C?.1, Q?.2, U?.32 (X1/CLK)
- new net: R?.2, U?.39 (VPA)
- new net: R?.2, U?.40 (BERR)
- new net: R?.2, U?.33 (BR)
- new net: R?.2, U?.36 (HALT)
- new net CTSA: J?.6 (Pin_6), U?.7 (IP0)
- new net CTSB: J?.6 (Pin_6), U?.4 (IP1)
- new net IACK: U?.8 (IN)
- new net RTSA: J?.2 (Pin_2), U?.29 (OP0)
- new net RTSB: J?.2 (Pin_2), U?.12 (OP1)
- new net RXDA: J?.4 (Pin_4), U?.31 (RXDA)
- new net RXDB: J?.4 (Pin_4), U?.10 (RXDB)
- new net SPICLK: J?.2 (Pin_2)
- new net SPICS: J?.1 (Pin_1)
- new net SPIMISO: J?.4 (Pin_4)
- new net SPIMOSI: J?.3 (Pin_3)
- new net TXDA: J?.5 (Pin_5), U?.30 (TXDA)
- new net TXDB: J?.5 (Pin_5), U?.11 (TXDB)
- new net ~{DTACK_DUART}: U?.7 (IN), U?.9 (DTACK)
- new net ~{DTACK}: U?.21 (I/O), U?.31 (DTACK)
- new net ~{DUARTSEL}: U?.21 (I/O), U?.3 (IN), U?.35 (CS)
- new net ~{IACK}: U?.1 (CLK/IN), U?.23 (I/O)
- new net ~{IOSEL}: U?.20 (I/O)
- new net ~{IPL0/2}: U?.42 (IPL0/2)
- no-connect marks 36 -> 25
Other:
- note added: "/RAM_WE = /RW * /DS /OE = RW * /DS /DTACK = ((RAMSEL + ROMSEL) * AS ) + (DUARTSEL * DTACK_DUART)"
- note added: "/ROMSL = IACK * /A17 * /A18 * /A19 /RAMSL = IACK * A17 * /A18 * /A19 /DUSL = IACK * A17 * A18 * /A19 /IOSL = IACK * A17 * A18 * A19 ROM (0x0000 - 0x1FFFF) RAM (0x20000 - 0x5FFFF) DUART (0x60000 - 0xDFFFF) IO (0xE0000 - 0xFFFFF)"
- note added: "Adddress Decoding"
- note added: "CS"
- note added: "Interrupt Handling"
- note added: "MISO"
- note added: "MOSI"
- note added: "SCK"
- note removed: "0x180000 start address"
- note removed: "AVR controls Serial, I2C and SPI as well as other simpler things. It can address 1024 (1k) bytes."
- note removed: "This connector has empty spaces so that the same bus can be used with processors that have 16 data lines and other control lines."
- moved on the sheet: C1, C2, C3, C4, C5, C6, D1, IC1, R10, R11, R12, R4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
