File: hardware/Steve 68k.kicad_sch (KiCad schematic)
At the start: 51 parts, among them IC1 MC68008FN8, J1 Power, J3 Debug, SW1 Reset, U1 74HC04, U2 74HC32, U3 74HC138, U4 74HC257, U5 AS6C4008-55PCN, U6 28C256, U8 Max705, X1 8Mhz

Commit message: V20221121
Parts:
- removed C11: 100uF, Capacitor_SMD:CP_Elec_4x5.4, symbol Device:C_Polarized
- removed C? (x2): 22pf, symbol Device:C
- removed C? (x5): .1uF, Capacitor_SMD:C_0603_1608Metric, symbol Device:C
- removed IC1: MC68008FN8, Package_LCC:PLCC-52_THT-Socket, symbol mc68k:MC68008FN8
- removed J1: Power, Connector_PinHeader_2.54mm:PinHeader_1x03_P2.54mm_Vertical, symbol Connector:Conn_01x03_Male
- removed J3: Debug, Connector_PinHeader_2.54mm:PinHeader_2x34_P2.54mm_Vertical, symbol Connector_Generic:Conn_02x34_Odd_Even
- removed J?: UART_A, rosco_m68k:1X06, symbol Connector:Conn_01x06_Male
- removed J?: UART_B, rosco_m68k:1X06, symbol Connector:Conn_01x06_Male
- removed J?: Conn_01x06, rosco_m68k:1X06, symbol Connector_Generic:Conn_01x06
- removed Q?: 3.6864MHz, Crystal:Crystal_HC49-4H_Vertical, symbol Device:Crystal
- removed R? (x4): 10k, Resistor_SMD:R_0603_1608Metric, symbol Device:R
- removed U1: 74HC04, Package_SO:SOIC-14_3.9x8.7mm_P1.27mm, symbol 74xx:74HC04
- removed U2: 74HC32, Package_SO:SOIC-14_3.9x8.7mm_P1.27mm, symbol 74xx:74LS32
- removed U3: 74HC138, Package_SO:SOIC-16_3.9x9.9mm_P1.27mm, symbol 74xx:74LS138
- removed U4: 74HC257, Package_SO:SOIC-16_3.9x9.9mm_P1.27mm, symbol 74xx:74LS257
- removed U5: AS6C4008-55PCN, Package_SO:SSOP-32_11.305x20.495mm_P1.27mm, symbol Memory_RAM:AS6C4008-55PCN
- removed U6: 28C256, Package_DIP:DIP-28_W15.24mm_Socket_LongPads, symbol Memory_EEPROM:28C256
- removed U? (x3): ATF22V10C, symbol rosco:ATF22V10C
- removed U?: 68681, symbol Interface:68681
- removed U?: 68008D, symbol CPU_NXP_68000:68008D
- added C10: 15pf, Capacitor_THT:C_Disc_D3.4mm_W2.1mm_P2.50mm, symbol Device:C
- added C11: 5pf, Capacitor_THT:C_Disc_D3.4mm_W2.1mm_P2.50mm, symbol Device:C
- added C12, C14, C15, C9: .1uF, Capacitor_THT:C_Disc_D3.4mm_W2.1mm_P2.50mm, symbol Device:C
- added C16: 470uF, Capacitor_THT:CP_Radial_D6.3mm_P2.50mm, symbol Device:C_Polarized
- added C17, C18, C19: 100uF, Capacitor_THT:CP_Radial_D5.0mm_P2.50mm, symbol Device:C_Polarized
- added D10: Data4, LED_THT:LED_D3.0mm_Clear, symbol Device:LED
- added D11: Data5, LED_THT:LED_D3.0mm_Clear, symbol Device:LED
- added D12: Data6, LED_THT:LED_D3.0mm_Clear, symbol Device:LED
- added D13: Data7, LED_THT:LED_D3.0mm_Clear, symbol Device:LED
- added D14: Data8, LED_THT:LED_D3.0mm_Clear, symbol Device:LED
- added D15: Data9, LED_THT:LED_D3.0mm_Clear, symbol Device:LED
- added D16: Data10, LED_THT:LED_D3.0mm_Clear, symbol Device:LED
- added D17: Data11, LED_THT:LED_D3.0mm_Clear, symbol Device:LED
- added D18: Data12, LED_THT:LED_D3.0mm_Clear, symbol Device:LED
- added D19: Data13, LED_THT:LED_D3.0mm_Clear, symbol Device:LED
- added D2: HALT, LED_THT:LED_D3.0mm_Clear, symbol Device:LED
- added D20: Data14, LED_THT:LED_D3.0mm_Clear, symbol Device:LED
- added D21: Data15, LED_THT:LED_D3.0mm_Clear, symbol Device:LED
- added D3: RUN, LED_THT:LED_D3.0mm_Clear, symbol Device:LED
- added D6: Data0, LED_THT:LED_D3.0mm_Clear, symbol Device:LED
- added D7: Data1, LED_THT:LED_D3.0mm_Clear, symbol Device:LED
- added D8: Data2, LED_THT:LED_D3.0mm_Clear, symbol Device:LED
- added D9: Data3, LED_THT:LED_D3.0mm_Clear, symbol Device:LED
- added J1: Conn_01x06_Male, Connector_PinHeader_2.54mm:PinHeader_1x06_P2.54mm_Vertical, symbol Connector:Conn_01x06_Male
- added J10: Debug 2, Connector_PinHeader_2.54mm:PinHeader_1x12_P2.54mm_Vertical, symbol Connector_Generic:Conn_01x12
- added J11: Duart IP, Connector_PinHeader_2.54mm:PinHeader_1x06_P2.54mm_Vertical, symbol Connector_Generic:Conn_01x06
- added J2, J5, J9: Conn_02x32_Odd_Even, Connector_PinSocket_2.54mm:PinSocket_2x32_P2.54mm_Vertical, symbol Connector_Generic:Conn_02x32_Odd_Even
- added J3, J4: Serial A, Connector_PinHeader_2.54mm:PinHeader_1x06_P2.54mm_Vertical, symbol Connector_Generic:Conn_01x06
- added J6: Data Bus, Connector_PinHeader_2.54mm:PinHeader_1x18_P2.54mm_Vertical, symbol Connector_Generic:Conn_01x18
- added J7: Debug, Connector_PinHeader_2.54mm:PinHeader_1x10_P2.54mm_Vertical, symbol Connector_Generic:Conn_01x10
- added J8: Duart OP, Connector_PinHeader_2.54mm:PinHeader_1x08_P2.54mm_Vertical, symbol Connector_Generic:Conn_01x08
- added Q1: 3.6864MHz, Crystal:Crystal_HC49-4H_Vertical, symbol Device:Crystal
- added R1: Rk7, Resistor_THT:R_Axial_DIN0207_L6.3mm_D2.5mm_P7.62mm_Horizontal, symbol Device:R
- added R13: 4k7, Resistor_THT:R_Axial_DIN0207_L6.3mm_D2.5mm_P7.62mm_Horizontal, symbol Device:R
- added R14, R15, R18, R19, R20, R21, R22, R23, R24, R25, R26, R27, R28, R29, R30, R31, R32, R33: 470, Resistor_THT:R_Axial_DIN0207_L6.3mm_D2.5mm_P7.62mm_Horizontal, symbol Device:R
- added R2, R3: 4K7, Resistor_THT:R_Axial_DIN0207_L6.3mm_D2.5mm_P7.62mm_Horizontal, symbol Device:R
- added U1, U3, U5: GAL16V8, Package_DIP:DIP-20_W7.62mm_Socket_LongPads, symbol Logic_Programmable:GAL16V8
- added U10, U9: 74LS373, Package_DIP:DIP-20_W7.62mm_Socket_LongPads, symbol 74xx:74LS373
- added U2: 68010D, Package_DIP:DIP-64_W22.86mm_Socket_LongPads, symbol CPU_NXP_68000:68010D
- added U4: 74LS148, Package_DIP:DIP-16_W7.62mm_Socket_LongPads, symbol 74xx:74LS148
- added U6: 68681, Package_DIP:DIP-40_W15.24mm_Socket_LongPads, symbol Interface:68681
- C1, C2, C3, C4, C5, C6, C7, C8: footprint Capacitor_SMD:C_0603_1608Metric -> Capacitor_THT:C_Disc_D3.4mm_W2.1mm_P2.50mm
- D1: footprint LED_SMD:LED_1206_3216Metric -> LED_THT:LED_D3.0mm_Clear
- R10, R4, R5, R6, R7, R8, R9: value 10k -> 4K7; footprint Resistor_SMD:R_0603_1608Metric -> Resistor_THT:R_Axial_DIN0207_L6.3mm_D2.5mm_P7.62mm_Horizontal
- R11: value 10k -> 4k7; footprint Resistor_SMD:R_0603_1608Metric -> Resistor_THT:R_Axial_DIN0207_L6.3mm_D2.5mm_P7.62mm_Horizontal
- R12: value 220 -> 470; footprint Resistor_SMD:R_0603_1608Metric -> Resistor_THT:R_Axial_DIN0207_L6.3mm_D2.5mm_P7.62mm_Horizontal
- U8: footprint Package_SO:SOIC-8_3.9x4.9mm_P1.27mm -> Package_DIP:DIP-8_W7.62mm_Socket_LongPads
Connections:
- net ~{DTACK_CPU} is gone; now on net VCC: R11.2
- net A1: now also J2.1 (Pin_1), J5.1 (Pin_1), J9.1 (Pin_1), U1.2 (I2), U2.29 (A1), U6.1 (RS1)
- net A10: now also J2.19 (Pin_19), J5.19 (Pin_19), J9.19 (Pin_19), U2.38 (A10)
- net A11: now also J2.21 (Pin_21), J5.21 (Pin_21), J9.21 (Pin_21), U2.39 (A11)
- net A12: now also J2.23 (Pin_23), J5.23 (Pin_23), J9.23 (Pin_23), U2.40 (A12)
- net A13: now also J2.25 (Pin_25), J5.25 (Pin_25), J9.25 (Pin_25), U2.41 (A13)
- net A14: now also J10.11 (Pin_11), J2.27 (Pin_27), J5.27 (Pin_27), J9.27 (Pin_27), U2.42 (A14), U5.8 (I8)
- net A15: now also J10.10 (Pin_10), J2.29 (Pin_29), J5.29 (Pin_29), J9.29 (Pin_29), U2.43 (A15), U5.7 (I7)
- net A16: now also J10.9 (Pin_9), J2.31 (Pin_31), J5.31 (Pin_31), J9.31 (Pin_31), U2.44 (A16), U5.6 (I6)
- net A17: now also J10.8 (Pin_8), J2.33 (Pin_33), J5.33 (Pin_33), J9.33 (Pin_33), U2.45 (A17), U5.5 (I5)
- net A18: now also J10.7 (Pin_7), J2.35 (Pin_35), J5.35 (Pin_35), J9.35 (Pin_35), U2.46 (A18), U5.4 (I4)
- net A19: now also J10.6 (Pin_6), J2.37 (Pin_37), J5.37 (Pin_37), J9.37 (Pin_37), U2.47 (A19), U3.1 (I1/CLK)
- net A2: now also J2.3 (Pin_3), J5.3 (Pin_3), J9.3 (Pin_3), U1.3 (I3), U2.30 (A2), U6.3 (RS2)
- net A20: now also J10.5 (Pin_5), J2.39 (Pin_39), J5.39 (Pin_39), J9.39 (Pin_39), U2.48 (A20), U3.2 (I2)
- net A21: now also J10.4 (Pin_4), J2.41 (Pin_41), J5.41 (Pin_41), J9.41 (Pin_41), U2.50 (A21), U3.3 (I3)
- net A3: now also J2.5 (Pin_5), J5.5 (Pin_5), J9.5 (Pin_5), U1.4 (I4), U2.31 (A3), U6.5 (RS3)
- net A4: now also J2.7 (Pin_7), J5.7 (Pin_7), J9.7 (Pin_7), U2.32 (A4), U6.6 (RS4)
- net A5: now also J2.9 (Pin_9), J5.9 (Pin_9), J9.9 (Pin_9), U2.33 (A5)
- net A6: now also J2.11 (Pin_11), J5.11 (Pin_11), J9.11 (Pin_11), U2.34 (A6)
- net A7: now also J2.13 (Pin_13), J5.13 (Pin_13), J9.13 (Pin_13), U2.35 (A7)
- net A8: now also J2.15 (Pin_15), J5.15 (Pin_15), J9.15 (Pin_15), U2.36 (A8)
- net A9: now also J2.17 (Pin_17), J5.17 (Pin_17), J9.17 (Pin_17), U2.37 (A9)
- net CLK: now also J2.4 (Pin_4), J5.4 (Pin_4), J9.4 (Pin_4), U1.1 (I1/CLK), U2.15 (CLK)
- net CTSA: now also J3.1 (Pin_1), U6.7 (IP0)
- net CTSB: now also J4.1 (Pin_1), U6.4 (IP1)
- net D0: now also J2.61 (Pin_61), J5.61 (Pin_61), J6.2 (Pin_2), J9.61 (Pin_61), U2.5 (D0), U6.25 (D0), U9.3 (D0)
- net D1: now also J2.63 (Pin_63), J5.63 (Pin_63), J6.3 (Pin_3), J9.63 (Pin_63), U2.4 (D1), U6.16 (D1), U9.4 (D1)
- net D2: now also J2.64 (Pin_64), J5.64 (Pin_64), J6.4 (Pin_4), J9.64 (Pin_64), U2.3 (D2), U6.24 (D2), U9.7 (D2)
- net D3: now also J2.62 (Pin_62), J5.62 (Pin_62), J6.5 (Pin_5), J9.62 (Pin_62), U2.2 (D3), U6.17 (D3), U9.8 (D3)
- net D4: now also J2.60 (Pin_60), J5.60 (Pin_60), J6.6 (Pin_6), J9.60 (Pin_60), U2.1 (D4), U6.23 (D4), U9.13 (D4)
- net D5: now also J2.58 (Pin_58), J5.58 (Pin_58), J6.7 (Pin_7), J9.58 (Pin_58), U2.64 (D5), U6.18 (D5), U9.14 (D5)
- net D6: now also J2.56 (Pin_56), J5.56 (Pin_56), J6.8 (Pin_8), J9.56 (Pin_56), U2.63 (D6), U6.22 (D6), U9.17 (D6)
- net D7: now also J2.54 (Pin_54), J5.54 (Pin_54), J6.9 (Pin_9), J9.54 (Pin_54), U2.62 (D7), U6.19 (D7), U9.18 (D7)
- net E: now also U2.20 (E)
- net FC0: now also J2.20 (Pin_20), J5.20 (Pin_20), J9.20 (Pin_20), U1.5 (I5), U2.28 (FC0)
- net FC1: now also J2.22 (Pin_22), J5.22 (Pin_22), J9.22 (Pin_22), U1.6 (I6), U2.27 (FC1)
- net FC2: now also J2.24 (Pin_24), J5.24 (Pin_24), J9.24 (Pin_24), U1.7 (I7), U2.26 (FC2)
- net GND: now also C2.1, C6.1, C10.2, C11.2, C12.2, C14.2, C15.2, C16.2, C17.2, C18.2, C19.2, C9.2, J1.2 (Pin_2), J10.1 (Pin_1), J10.12 (Pin_12), J11.6 (Pin_6), J2.6 (Pin_6), J3.6 (Pin_6), J4.6 (Pin_6), J5.6 (Pin_6), J6.1 (Pin_1), J6.18 (Pin_18), J7.1 (Pin_1), J7.10 (Pin_10), J8.8 (Pin_8), J9.6 (Pin_6), R18.1, R19.1, R20.1, R21.1, R22.1, R23.1, R24.1, R25.1, R26.1, R27.1, R28.1, R29.1, R30.1, R31.1, R32.1, R33.1, U1.10 (GND), U10.1 (OE), U10.10 (GND), U2.16 (GND), U2.53 (GND), U3.10 (GND), U4.10 (IO), U4.5 (EI), U4.8 (GND), U5.10 (GND), U6.20 (GND), U9.1 (OE), U9.10 (GND); no longer C2.2, C6.2
- net RTSA: now also J3.5 (Pin_5), U6.29 (OP0)
- net RTSB: now also J4.5 (Pin_5), U6.12 (OP1)
- net RXDA: now also J3.3 (Pin_3), U6.31 (RXDA)
- net RXDB: now also J4.3 (Pin_3), U6.10 (RXDB)
- net R~{W}: now also J2.59 (Pin_59), J5.59 (Pin_59), J7.2 (Pin_2), J9.59 (Pin_59), U2.9 (R/W), U5.3 (I3), U6.8 (R/W)
- net TXDA: now also J3.2 (Pin_2), U6.30 (TXDA)
- net TXDB: now also J4.2 (Pin_2), U6.11 (TXDB)
- net VCC: now also C2.2, C6.2, D1.1 (K), C12.1, C14.1, C15.1, C16.1, C17.1, C18.1, C19.1, C9.1, D2.1 (K), D3.1 (K), J1.1 (Pin_1), J11.1 (Pin_1), J2.2 (Pin_2), J5.2 (Pin_2), J8.1 (Pin_1), J9.2 (Pin_2), R1.1, R13.2, R2.1, R3.1, U1.20 (VCC), U10.20 (VCC), U2.14 (VCC), U2.49 (VCC), U3.20 (VCC), U4.11 (I1), U4.16 (VCC), U4.4 (I7), U5.20 (VCC), U6.40 (VCC), U9.20 (VCC); no longer C2.1, C6.1, D1.2 (A), R11.1
- net ~{AS}: now also J2.47 (Pin_47), J5.47 (Pin_47), J7.4 (Pin_4), J9.47 (Pin_47), U2.6 (AS), U3.6 (I6); no longer R10.2
- net ~{BERR}: now also J2.49 (Pin_49), J5.49 (Pin_49), J9.49 (Pin_49), R2.2, U2.22 (BERR); no longer R4.2
- net ~{BGACK}: now also R5.2, J2.53 (Pin_53), J5.53 (Pin_53), J9.53 (Pin_53), U2.12 (BGACK); no longer R8.2
- net ~{BG}: now also J2.51 (Pin_51), J5.51 (Pin_51), J9.51 (Pin_51), U2.11 (BG)
- net ~{BR}: now also R4.2, J2.55 (Pin_55), J5.55 (Pin_55), J9.55 (Pin_55), U2.13 (BR); no longer R7.2
- net ~{DTACK}: now also J2.57 (Pin_57), J5.57 (Pin_57), J7.3 (Pin_3), J9.57 (Pin_57), U2.10 (DTACK), U5.18 (IO2), U6.9 (DTACK)
- net ~{HALT}: now also J2.16 (Pin_16), J5.16 (Pin_16), J7.9 (Pin_9), J9.16 (Pin_16), R1.2, R14.1, U1.8 (I8), U2.17 (HALT); no longer R6.2
- net ~{IACK}: now also J2.10 (Pin_10), J5.10 (Pin_10), J7.8 (Pin_8), J9.10 (Pin_10), U1.19 (IO1), U6.37 (IACK)
- net ~{IOSEL}: now also J2.12 (Pin_12), J5.12 (Pin_12), J7.7 (Pin_7), J9.12 (Pin_12), U3.19 (IO1), U5.9 (I9)
- net ~{IPL0}: now also U2.25 (IPL0), U4.9 (S0)
- net ~{IPL1}: now also U2.24 (IPL1), U4.7 (S1)
- net ~{IPL2}: now also U2.23 (IPL2), U4.6 (S2)
- net ~{RESET}: now also J2.36 (Pin_36), J5.36 (Pin_36), J9.36 (Pin_36), U1.9 (I9), U2.18 (RESET), U3.9 (I9), U6.34 (RESET)
- net ~{VPA}: now also R3.2, U2.21 (VPA); no longer R5.2
- net at R12.2: now also D1.2 (A); no longer D1.1 (K)
- net ~{DTACK_AVR} renamed ~{IRQ5}
- net ~{IRQ5}: now also J2.26 (Pin_26), J5.26 (Pin_26), J9.26 (Pin_26), U4.2 (I5)
- new net: D18.1 (K), R30.2
- new net: D18.2 (A), U10.12 (O4)
- new net: D11.1 (K), R23.2
- new net: D11.2 (A), U9.15 (O5)
- new net: D21.1 (K), R33.2
- new net: D21.2 (A), U10.19 (O7)
- new net: D16.1 (K), R28.2
- new net: D16.2 (A), U10.6 (O2)
- new net: D17.1 (K), R29.2
- new net: D17.2 (A), U10.9 (O3)
- new net: D6.1 (K), R18.2
- new net: D6.2 (A), U9.2 (O0)
- new net: D12.1 (K), R24.2
- new net: D19.2 (A), U10.15 (O5)
- new net: D20.2 (A), U10.16 (O6)
- new net: D14.2 (A), U10.2 (O0)
- new net: D15.2 (A), U10.5 (O1)
- new net: D9.1 (K), R21.2
- new net: D9.2 (A), U9.9 (O3)
- new net: D8.1 (K), R20.2
- new net: D8.2 (A), U9.6 (O2)
- new net: D15.1 (K), R27.2
- new net: D13.1 (K), R25.2
- new net: D14.1 (K), R26.2
- new net: D3.2 (A), R15.2
- new net: D20.1 (K), R32.2
- new net: C10.1, Q1.2, U6.32 (X1/CLK)
- new net: C11.1, Q1.1, U6.33 (X2)
- new net: D10.2 (A), U9.12 (O4)
- new net: D12.2 (A), U9.16 (O6)
- new net: D13.2 (A), U9.19 (O7)
- new net: D7.2 (A), U9.5 (O1)
- new net: D19.1 (K), R31.2
- new net: D10.1 (K), R22.2
- new net: D7.1 (K), R19.2
- new net: D2.2 (A), R14.2
- new net A22: J10.3 (Pin_3), J2.43 (Pin_43), J5.43 (Pin_43), J9.43 (Pin_43), U2.51 (A22), U3.4 (I4)
- new net A23: J10.2 (Pin_2), J2.45 (Pin_45), J5.45 (Pin_45), J9.45 (Pin_45), U2.52 (A23), U3.5 (I5)
- new net D10: J2.48 (Pin_48), J5.48 (Pin_48), J6.12 (Pin_12), J9.48 (Pin_48), U10.7 (D2), U2.59 (D10)
- new net D11: J2.46 (Pin_46), J5.46 (Pin_46), J6.13 (Pin_13), J9.46 (Pin_46), U10.8 (D3), U2.58 (D11)
- new net D12: J2.44 (Pin_44), J5.44 (Pin_44), J6.14 (Pin_14), J9.44 (Pin_44), U10.13 (D4), U2.57 (D12)
- new net D13: J2.42 (Pin_42), J5.42 (Pin_42), J6.15 (Pin_15), J9.42 (Pin_42), U10.14 (D5), U2.56 (D13)
- new net D14: J2.40 (Pin_40), J5.40 (Pin_40), J6.16 (Pin_16), J9.40 (Pin_40), U10.17 (D6), U2.55 (D14)
- new net D15: J2.38 (Pin_38), J5.38 (Pin_38), J6.17 (Pin_17), J9.38 (Pin_38), U10.18 (D7), U2.54 (D15)
- new net D8: J2.52 (Pin_52), J5.52 (Pin_52), J6.10 (Pin_10), J9.52 (Pin_52), U10.3 (D0), U2.61 (D8)
- new net D9: J2.50 (Pin_50), J5.50 (Pin_50), J6.11 (Pin_11), J9.50 (Pin_50), U10.4 (D1), U2.60 (D9)
- new net IP2: J11.2 (Pin_2), U6.36 (IP2)
- new net IP3: J11.3 (Pin_3), U6.2 (IP3)
- new net IP4: J11.4 (Pin_4), U6.39 (IP4)
- new net IP5: J11.5 (Pin_5), U6.38 (IP5)
- new net OP2: J8.2 (Pin_2), U6.28 (OP2)
- new net OP3: J8.3 (Pin_3), U6.13 (OP3)
- new net OP4: J8.4 (Pin_4), U6.27 (OP4)
- new net OP5: J8.5 (Pin_5), U6.14 (OP5)
- new net OP6: J8.6 (Pin_6), U6.26 (OP6)
- new net OP7: J8.7 (Pin_7), U6.15 (OP7)
- new net STATUSHI: R13.1, U10.11 (LE), U5.16 (IO4)
- new net STATUSLO: R11.1, U5.17 (I03), U9.11 (LE)
- new net ~{IRQ2}: R6.2, U4.12 (I2), U6.21 (IRQ)
- new net ~{IRQ3}: J2.14 (Pin_14), J5.14 (Pin_14), J9.14 (Pin_14), R7.2, U4.13 (I3)
- new net ~{IRQ4}: J2.18 (Pin_18), J5.18 (Pin_18), J9.18 (Pin_18), R8.2, U4.1 (I4)
- new net ~{IRQ6}: J2.30 (Pin_30), J5.30 (Pin_30), J9.30 (Pin_30), R10.2, U4.3 (I6)
- new net ~{LDS}: J2.32 (Pin_32), J5.32 (Pin_32), J7.5 (Pin_5), J9.32 (Pin_32), U2.8 (LDS), U3.8 (I8), U5.2 (I2)
- new net ~{RUN}: R15.1, U3.18 (IO2)
- new net ~{UARTSEL}: U5.19 (IO1), U6.35 (CS)
- new net ~{UDS}: J2.34 (Pin_34), J5.34 (Pin_34), J7.6 (Pin_6), J9.34 (Pin_34), U2.7 (UDS), U3.7 (I7), U5.1 (I1/CLK)
- new net ~{VMA}: J2.28 (Pin_28), J5.28 (Pin_28), J9.28 (Pin_28), U2.19 (VMA)
- new net ~{VPA: J2.8 (Pin_8), J5.8 (Pin_8), J9.8 (Pin_8)
- no-connect marks 25 -> 32
Other:
- note added: "/IACK = /FC0 * /FC1 */FC2 * /A1 * /A2 * A3"
- note added: "/IOSEL = A19 * A20 * A21 * A22 * A23 * /AS /BOOT = GND /RUN = GND"
- note added: "/UARTSEL = /IOSEL * /LDS * /A18 * /A17 * /A16 * /A15 * /A14"
- note removed: "/RAM_WE = /RW * /DS /OE = RW * /DS /DTACK = ((RAMSEL + ROMSEL) * AS ) + (DUARTSEL * DTACK_DUART)"
- note removed: "/ROMSL = IACK * /A17 * /A18 * /A19 /RAMSL = IACK * A17 * /A18 * /A19 /DUSL = IACK * A17 * A18 * /A19 /IOSL = IACK * A17 * A18 * A19 ROM (0x0000 - 0x1FFFF) RAM (0x20000 - 0x5FFFF) DUART (0x60000 - 0xDFFFF) IO (0xE0000 - 0xFFFFF)"
- note removed: "0x0000-0x7FFF"
- note removed: "0x10000-"
- note removed: "0x8000-0xFFFF"
- note removed: "Adddress Decoding"
- note removed: "CS"
- note removed: "IF AVRSEL is LOW then DTACK will be DTACK_AVR otherwise it's the AS"
- note removed: "Interrupt Handling"
- note removed: "MISO"
- note removed: "MOSI"
- note removed: "SCK"
- note removed: "Will set OE low if RW is HIGH (READ) and DS is LOW"
- note removed: "Will set RAM_WE LOW when RW is LOW (WRITE) AND DS is LOW"
- moved on the sheet: C1, C4, C5, D1, R12, SW1, U8, X1
