File: hardware/Steve 68k.kicad_pcb (KiCad board)
At the start: 2 copper layers, 99 x 98.9 mm, 46 parts, among them IC1 MC68008FN8, J1 Conn_02x32_Odd_Even, J2 Serial 1, J3 Serial 2, J4 Conn_01x03_Male, SW1 Reset, U1 74LS32, U2 28C256, U3 GAL16V8, U4 74HC04, U5 MC68681FN, U7 AS6C4008-55PCN, U8 Max705, X1 CXO_DIP8, X2 1.8432 Mhz

Commit message: Latest version sent for fab
Parts:
- removed REF**: OSHW-Logo2_9.8x8mm_SilkScreen, Symbol:OSHW-Logo2_9.8x8mm_SilkScreen
- removed X2: 1.8432 Mhz, Oscillator:Oscillator_DIP-14
- added C13: 100uF, Capacitor_SMD:CP_Elec_4x5.4, F.Cu at (133.5, 95.8)
- added C5: 12pf, Capacitor_SMD:C_0603_1608Metric, F.Cu at (139.3, 39.2)
- added D6: PWR, LED_SMD:LED_1206_3216Metric, F.Cu at (135.1, 102.9)
- added D7: ERR, LED_SMD:LED_1206_3216Metric, F.Cu at (156.6, 65.9)
- added J6: Serial 2, Connector_PinSocket_2.54mm:PinSocket_1x06_P2.54mm_Vertical, F.Cu at (150.6, 47.9)
- added R14: 10k, Resistor_SMD:R_0603_1608Metric, F.Cu at (92.6, 103.7)
- added R15: 10k, Resistor_SMD:R_0603_1608Metric, F.Cu at (92.6, 108.1)
- added R16: 10k, Resistor_SMD:R_0603_1608Metric, F.Cu at (92.6, 112.4)
- added R17: 220, Resistor_SMD:R_0603_1608Metric, F.Cu at (130.3, 102.9)
- added R18: 220, Resistor_SMD:R_0603_1608Metric, F.Cu at (152.0, 65.9)
- added U6: L7805, Package_TO_SOT_THT:TO-220-3_Horizontal_TabUp, F.Cu at (159.6, 93.9)
- added Y1: 3.6864, Crystal:Crystal_HC49-U_Vertical, F.Cu at (139.3, 49.8)
- C9: value .1uF -> 12pf
- J2: value Serial 1 -> 5V Input; footprint Connector_PinHeader_2.54mm:PinHeader_1x04_P2.54mm_Vertical -> Connector_BarrelJack:BarrelJack_Horizontal
- J3: value Serial 2 -> Serial 1; footprint Connector_PinHeader_2.54mm:PinHeader_1x04_P2.54mm_Vertical -> Connector_PinSocket_2.54mm:PinSocket_1x06_P2.54mm_Vertical
- J4: value Conn_01x03_Male -> CLK Select
- U4: footprint Package_SO:SOIC-14_3.9x8.7mm_P1.27mm -> Package_SO:SOIC-14W_7.5x9mm_P1.27mm
- U8: footprint Package_DIP:DIP-8_W7.62mm_Socket_LongPads -> Package_SO:SOIC-8_3.9x4.9mm_P1.27mm
- moved J2 55.2 mm to (148.7, 112.1), turned to 180 degrees
- moved C10 35.8 mm to (109.6, 115.1)
- moved U1 34.6 mm to (114.6, 112.0), turned to 0 degrees
- moved U4 32.3 mm to (114.5, 99.4), turned to 0 degrees
- moved U8 28.4 mm to (126.2, 112.9), turned to 0 degrees
- moved C4 24.3 mm to (126.2, 107.9), turned to 0 degrees
- moved C11 22.2 mm to (114.7, 92.4), turned to 0 degrees
- moved C9 16.9 mm to (139.3, 55.4)
- moved C12 15.8 mm to (134.4, 112.0)
- moved SW1 15.7 mm to (137.3, 109.7)
- moved C7 11.9 mm to (109.2, 78.7), turned to 90 degrees
- moved U7 6.36 mm to (122.3, 78.8), turned to 90 degrees
- moved J3 4.33 mm to (158.9, 47.9)
- moved C1 0.98 mm to (100.6, 89.0)
- moved U3 0.98 mm to (96.7, 92.9)
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Connections:
- net /OP0 renamed /RTSA
- net /OP2 renamed /RTSB
- C9 pad 1: VCC -> GND
- C9 pad 2: GND -> /68681_X2
- IC1 pad 46: /68681_Int -> /~{IPL2}
- J1 pad 52: /68681_Int -> /~{IPL2}
- J2 pad 1: GND -> Net-(J2-Pad1)
- J2 pad 2: /RxDA -> Net-(C13-Pad2)
- J2 pad 3: /TxDA -> (no net)
- J3 pad 1: GND -> /DTRA
- J3 pad 2: /RxDB -> /TxDA
- J3 pad 3: /TxDB -> /RxDA
- R2 pad 2: /68681_Int -> /~{IPL2}
- U3 pad 1: /CLK -> /A18
- U3 pad 11: GND -> /A17
- U3 pad 17: unconnected-(U3-Pad17) -> /ERROR
- U3 pad 7: /DTACK_I2C -> /~{DTACK_I2C}
- U5 pad 36: /UART_CLK -> /68681_X1
- U5 pad 37: unconnected-(U5-Pad37) -> /68681_X2
- U5 pad 5: /IP1 -> /CTSB
- U5 pad 8: /IP0 -> /CTSA
Routing:
- net /~{IPL2}: track 0.00 -> 106.5 mm, vias 0 -> 1
- net VCC: track 401.0 -> 505.6 mm, vias 5 -> 4
- net /~{DS}: track 164.6 -> 84.3 mm
- net Net-(C13-Pad2): track 0.00 -> 64.0 mm
- net GND: track 504.1 -> 440.8 mm, vias 4 -> 21
- net /ERROR: track 0.00 -> 63.2 mm
- net /R~{W}: track 159.6 -> 104.5 mm, vias 2 -> 5
- net /CTSA: track 0.00 -> 52.1 mm
- net /CTSB: track 0.00 -> 44.4 mm
- net /A10: track 133.0 -> 177.0 mm, vias 1 -> 0
- net Net-(R9-Pad1): track 13.9 -> 53.6 mm
- net Net-(R5-Pad1): track 16.0 -> 51.7 mm
- net /~{USERSEL}: track 119.4 -> 85.2 mm, vias 1 -> 0
- net Net-(R7-Pad1): track 20.3 -> 53.1 mm
- net /~{I2CSEL}: track 95.2 -> 63.2 mm
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- added copper zone on F.Cu, net GND
Other:
- board text added: "ERROR"
- board text added: "Ex CLK"
- board text added: "V20220621"
- board text added: "~{DTUSER}"
- board text removed: "Ext CLK"
- board text removed: "RX"
- board text removed: "TX"
- board text removed: "V20220601"
- board text removed: "VCC"

Commit message: Board Schematic image and PDF
Routing:
- net Net-(C13-Pad2): track 64.0 -> 62.3 mm
- net /CTSA: track 52.1 -> 52.8 mm
Changed lines of the file:
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@@
   (segment (start 105.8177 108.1786) (end 108.3448 105.6515) (width 0.25) (layer "F.Cu") (net 77))
   (via (at 130.0362 96.6541) (size 0.8) (drill 0.4) (layers "F.Cu" "B.Cu") (net 77))
+  (segment (start 130.429 95.645417) (end 130.429 96.597) (width 0.25) (layer "B.Cu") (net 77))
   (segment (start 135.9339 127.2012) (end 136.7418 128.0091) (width 0.25) (layer "B.Cu") (net 77))
-  (segment (start 130.48 51.8451) (end 130.48 96.648) (width 0.25) (layer "B.Cu") (net 77))
+  (segment (start 130.47912 51.84598) (end 130.47912 95.595297) (width 0.25) (layer "B.Cu") (net 77))
+  (segment (start 131.5212 47.244) (end 132.5961 48.3189) (width 0.25) (layer "B.Cu") (net 77))
   (segment (start 136.7418 128.0091) (end 137.1092 128.0091) (width 0.25) (layer "B.Cu") (net 77))
-  (segment (start 131.5212 47.244) (end 132.5961 48.3189) (width 0.25) (layer "B.Cu") (net 77))
-  (segment (start 131.7432 51.054) (end 131.2711 51.054) (width 0.25) (layer "B.Cu") (net 77))
   (segment (start 135.9339 102.1019) (end 135.9339 127.2012) (width 0.25) (layer "B.Cu") (net 77))
+  (segment (start 131.2711 51.054) (end 130.47912 51.84598) (width 0.25) (layer "B.Cu") (net 77))
+  (segment (start 132.5961 50.2011) (end 131.7432 51.054) (width 0.25) (layer "B.Cu") (net 77))
   (segment (start 130.0423 96.648) (end 130.0362 96.6541) (width 0.25) (layer "B.Cu") (net 77))
-  (segment (start 132.5961 50.2011) (end 131.7432 51.054) (width 0.25) (layer "B.Cu") (net 77))
+  (segment (start 130.429 96.597) (end 130.48 96.648) (width 0.25) (layer "B.Cu") (net 77))
   (segment (start 137.1092 129.1844) (end 137.1092 128.0091) (width 0.25) (layer "B.Cu") (net 77))
   (segment (start 130.48 96.648) (end 130.0423 96.648) (width 0.25) (layer "B.Cu") (net 77))
+  (segment (start 131.7432 51.054) (end 131.2711 51.054) (width 0.25) (layer "B.Cu") (net 77))
   (segment (start 132.5961 48.3189) (end 132.5961 50.2011) (width 0.25) (layer "B.Cu") (net 77))
   (segment (start 130.48 96.648) (end 135.9339 102.1019) (width 0.25) (layer "B.Cu") (net 77))
-  (segment (start 131.2711 51.054) (end 130.48 51.8451) (width 0.25) (layer "B.Cu") (net 77))
+  (segment (start 130.47912 95.595297) (end 130.429 95.645417) (width 0.25) (layer "B.Cu") (net 77))
   (segment (start 140.0432 54.3224) (end 139.8897 54.1689) (width 0.25) (layer "F.Cu") (net 83))
   (segment (start 131.5212 49.784) (end 139.2682 49.784) (width 0.25) (layer "F.Cu") (net 83))
@@
   (segment (start 139.2936 49.7586) (end 139.8897 50.3547) (width 0.25) (layer "B.Cu") (net 83))
   (segment (start 139.8897 50.3547) (end 139.8897 54.1689) (width 0.25) (layer "B.Cu") (net 83))
-  (segment (start 150.734403 102.59828) (end 159.14848 102.59828) (width 0.25) (layer "F.Cu") (net 85))
+  (segment (start 139.2174 106.6546) (end 146.678083 106.6546) (width 0.25) (layer "F.Cu") (net 85))
+  (segment (start 150.734403 102.59828) (end 158.1912 102.59828) (width 0.25) (layer "F.Cu") (net 85))
+  (segment (start 158.1912 97.7998) (end 159.598 96.393) (width 0.25) (layer "F.Cu") (net 85))
+  (segment (start 133.5278 97.6088) (end 135.0334 99.1144) (width 0.25) (layer "F.Cu") (net 85))
+  (segment (start 136.5026 103.9398) (end 139.2174 106.6546) (width 0.25) (layer "F.Cu") (net 85))
+  (segment (start 158.1912 102.59828) (end 158.1912 97.7998) (width 0.25) (layer "F.Cu") (net 85))
+  (segment (start 135.0334 99.1144) (end 136.5026 99.1144) (width 0.25) (layer "F.Cu") (net 85))
+  (segment (start 136.5026 99.1144) (end 136.5026 102.9208) (width 0.25) (layer "F.Cu") (net 85))
   (segment (start 136.5026 99.1144) (end 136.5026 103.9398) (width 0.25) (layer "F.Cu") (net 85))
-  (segment (start 159.598 97.65598) (end 159.598 96.393) (width 0.25) (layer "F.Cu") (net 85))
-  (segment (start 159.021541 97.65598) (end 159.598 97.65598) (width 0.25) (layer "F.Cu") (net 85))
-  (segment (start 159.14848 102.59828) (end 159.14848 100.21002) (width 0.25) (layer "F.Cu") (net 85))
-  (segment (start 139.2174 106.6546) (end 146.678083 106.6546) (width 0.25) (layer "F.Cu") (net 85))
-  (segment (start 159.14848 100.21002) (end 159.021541 100.21002) (width 0.25) (layer "F.Cu") (net 85))
-  (segment (start 133.5278 97.6088) (end 135.0334 99.1144) (width 0.25) (layer "F.Cu") (net 85))
-  (segment (start 158.27348 99.461959) (end 158.27348 98.404041) (width 0.25) (layer "F.Cu") (net 85))
-  (segment (start 135.0334 99.1144) (end 136.5026 99.1144) (width 0.25) (layer "F.Cu") (net 85))
-  (segment (start 136.5026 103.9398) (end 139.2174 106.6546) (width 0.25) (layer "F.Cu") (net 85))
-  (segment (start 136.5026 99.1144) (end 136.5026 102.9208) (width 0.25) (layer "F.Cu") (net 85))
-  (segment (start 159.021541 100.21002) (end 158.27348 99.461959) (width 0.25) (layer "F.Cu") (net 85))
-  (segment (start 158.27348 98.404041) (end 159.021541 97.65598) (width 0.25) (layer "F.Cu") (net 85))
   (segment (start 146.678083 106.6546) (end 150.734403 102.59828) (width 0.25) (layer "F.Cu") (net 85))
   (segment (start 154.9146 112.1587) (end 154.9146 105.469879) (width 0.25) (layer "B.Cu") (net 85))
@@
   (segment (start 120.0154 74.6501) (end 120.0154 87.5005) (width 0.25) (layer "B.Cu") (net 106))
   (segment (start 128.3139 124.7765) (end 128.3139 127.2012) (width 0.25) (layer "B.Cu") (net 106))
-  (segment (start 117.3343 46.1909) (end 151.0715 46.1909) (width 0.25) (layer "F.Cu") (net 111))
-  (segment (start 116.2812 47.244) (end 117.3343 46.1909) (width 0.25) (layer "F.Cu") (net 111))
-  (segment (start 156.695 52.4825) (end 158.4669 54.2544) (width 0.25) (layer "F.Cu") (net 111))
-  (segment (start 159.2952 56.8891) (end 158.9278 56.8891) (width 0.25) (layer "F.Cu") (net 111))
-  (segment (start 151.0715 46.1909) (end 156.695 51.8144) (width 0.25) (layer "F.Cu") (net 111))
-  (segment (start 158.9278 58.0644) (end 158.9278 56.8891) (width 0.25) (layer "F.Cu") (net 111))
-  (segment (start 156.695 51.8144) (end 156.695 52.4825) (width 0.25) (layer "F.Cu") (net 111))
-  (segment (start 160.1031 56.0812) (end 159.2952 56.8891) (width 0.25) (layer "F.Cu") (net 111))
-  (segment (start 159.4024 54.2544) (end 160.1031 54.9551) (width 0.25) (layer "F.Cu") (net 111))
   (segment (start 160.1031 54.9551) (end 160.1031 56.0812) (width 0.25) (layer "F.Cu") (net 111))
   (segment (start 158.4669 54.2544) (end 159.4024 54.2544) (width 0.25) (layer "F.Cu") (net 111))
+  (segment (start 159.4024 54.2544) (end 160.1031 54.9551) (width 0.25) (layer "F.Cu") (net 111))
+  (segment (start 117.3343 46.1909) (end 152.2105 46.1909) (width 0.25) (layer "F.Cu") (net 111))
+  (segment (start 156.695 52.4825) (end 158.4669 54.2544) (width 0.25) (layer "F.Cu") (net 111))
+  (segment (start 116.2812 47.244) (end 117.3343 46.1909) (width 0.25) (layer "F.Cu") (net 111))
+  (segment (start 152.2105 46.1909) (end 156.695 50.6754) (width 0.25) (layer "F.Cu") (net 111))
+  (segment (start 160.1031 56.0812) (end 159.2952 56.8891) (width 0.25) (layer "F.Cu") (net 111))
+  (segment (start 156.695 50.6754) (end 156.695 52.4825) (width 0.25) (layer "F.Cu") (net 111))
+  (segment (start 158.9278 56.8891) (end 158.9278 58.0644) (width 0.25) (layer "F.Cu") (net 111))
+  (segment (start 159.2952 56.8891) (end 158.9278 56.8891) (width 0.25) (layer "F.Cu") (net 111))
   (segment (start 149.4209 56.0812) (end 150.2288 56.8891) (width 0.25) (layer "F.Cu") (net 113))
   (segment (start 151.776 53.522) (end 151.0436 54.2544) (width 0.25) (layer "F.Cu") (net 113))

Commit message: V20220905 sent for fab
Parts:
- removed C13: 100uF, Capacitor_SMD:CP_Elec_4x5.4
- removed C15: 10uF, Capacitor_SMD:CP_Elec_4x5.4
- removed D3: RAM, LED_SMD:LED_1206_3216Metric
- removed D4: UART, LED_SMD:LED_1206_3216Metric
- removed D5: USER, LED_SMD:LED_1206_3216Metric
- removed D6: PWR, LED_SMD:LED_1206_3216Metric
- removed D7: ERR, LED_SMD:LED_1206_3216Metric
- removed J6: Serial 2, Connector_PinSocket_2.54mm:PinSocket_1x06_P2.54mm_Vertical
- removed R14, R15, R16: 10k, Resistor_SMD:R_0603_1608Metric
- removed R17, R18: 220, Resistor_SMD:R_0603_1608Metric
- removed the U6 at (159.6, 93.9)
- removed Y1: 3.6864, Crystal:Crystal_HC49-U_Vertical
- added J5: Serial 1, Connector_PinSocket_2.54mm:PinSocket_1x06_P2.54mm_Vertical, F.Cu at (157.0, 43.9)
- added U2: 74HC32, Package_SO:SOIC-14_3.9x8.7mm_P1.27mm, F.Cu at (105.9, 109.4)
- C1: value .1uF -> 100nf
- C11: value .1uF -> 100uF; footprint Capacitor_SMD:C_0603_1608Metric -> Capacitor_SMD:CP_Elec_4x5.4
- C12: value 100nf -> .1uF
- C5, C9: value 12pf -> .1uF
- D1: value I2C -> PWR LED
- D2: value ROM -> BLINK LED
- J1: value Conn_02x32_Odd_Even -> Power; footprint Connector_PinHeader_2.54mm:PinHeader_2x32_P2.54mm_Vertical -> Connector_PinHeader_2.54mm:PinHeader_1x03_P2.54mm_Vertical
- J2: value 5V Input -> I2C; footprint Connector_BarrelJack:BarrelJack_Horizontal -> Connector_PinSocket_2.54mm:PinSocket_1x04_P2.54mm_Vertical
- J3: value Serial 1 -> Debug; footprint Connector_PinSocket_2.54mm:PinSocket_1x06_P2.54mm_Vertical -> Connector_PinHeader_2.54mm:PinHeader_2x34_P2.54mm_Vertical
- J4: value CLK Select -> ICSP; footprint Connector_PinHeader_2.54mm:PinHeader_1x03_P2.54mm_Vertical -> Connector_PinSocket_2.54mm:PinSocket_2x03_P2.54mm_Vertical
- R12, R13: value 10k -> 220
- R5, R6, R7, R8, R9: value 220 -> 10k
- U1: value 74LS32 -> 74HC04
- U3: value GAL16V8 -> 74HC138; footprint Package_DIP:DIP-20_W7.62mm_Socket_LongPads -> Package_SO:SOIC-16_3.9x9.9mm_P1.27mm
- U4: value 74HC04 -> 74HC257; footprint Package_SO:SOIC-14W_7.5x9mm_P1.27mm -> Package_SO:SOIC-16_3.9x9.9mm_P1.27mm
- U5: value MC68681FN -> AS6C4008-55PCN; footprint Package_LCC:PLCC-44_THT-Socket -> Package_SO:SSOP-32_11.305x20.495mm_P1.27mm
- U7: value AS6C4008-55PCN -> ATmega1284P-P; footprint Package_SO:SSOP-32_11.305x20.495mm_P1.27mm -> Package_DIP:DIP-40_W15.24mm
- X1: value CXO_DIP8 -> 8Mhz
- moved J3 117.9 mm to (72.1, 127.8), turned to 90 degrees
- moved J1 88.2 mm to (157.5, 111.8), turned to 0 degrees
- moved C12 72.7 mm to (131.6, 39.4), turned to 0 degrees
- moved C6 67.0 mm to (131.3, 102.4), turned to 0 degrees
- moved R12 64.9 mm to (144.8, 115.3), turned to 180 degrees
- moved C9 64.4 mm to (95.2, 102.4)
- moved C5 63.3 mm to (142.5, 102.4)
- moved R6 59.6 mm to (100.3, 56.6), turned to 180 degrees
- moved R5 58.6 mm to (100.3, 54.9), turned to 180 degrees
- moved J4 56.3 mm to (115.6, 76.0)
- moved R10 55.4 mm to (125.0, 108.2)
- moved R11 53.6 mm to (125.0, 110.0)
- moved R8 53.6 mm to (100.3, 60.2), turned to 180 degrees
- moved R7 53.0 mm to (100.3, 58.4), turned to 180 degrees
- moved C1 48.1 mm to (146.8, 102.4)
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- renumbered U2 to U6
Connections:
- C1 pad 1: VCC -> Net-(C1-Pad1)
- C12 pad 1: Net-(C12-Pad1) -> VCC
- C5 pad 1: GND -> VCC
- C5 pad 2: /68681_X1 -> GND
- C9 pad 1: GND -> VCC
- C9 pad 2: /68681_X2 -> GND
- D1 pad 1: GND -> Net-(D1-Pad1)
- D1 pad 2: Net-(D1-Pad2) -> VCC
- D2 pad 1: GND -> Net-(D2-Pad1)
- IC1 pad 43: /68681_Int -> /~{VPA}
- J1 pad 1: /A0 -> VCC
- J1 pad 2: /A1 -> unconnected-(J1-Pad2)
- J1 pad 3: /A2 -> GND
- J2 pad 1: Net-(J2-Pad1) -> VCC
- J2 pad 2: Net-(C13-Pad2) -> GND
- J2 pad 3: (no net) -> /SDA
- J3 pad 1: /DTRA -> GND
- J3 pad 2: /TxDA -> GND
- J3 pad 3: /RxDA -> /A0
- J3 pad 4: VCC -> /A1
- J3 pad 5: /CTSA -> /A2
- J3 pad 6: GND -> /A3
- J4 pad 1: /CLK_ONBOARD -> /MISO
- J4 pad 2: /CLK -> /SCK
- J4 pad 3: /CLK_EXTERNAL -> /~{RESET}
- R10 pad 2: /~{HALT} -> /~{AS}
- R11 pad 2: /~{BERR} -> /~{DTACK_CPU}
- R12 pad 1: VCC -> GND
- R12 pad 2: /~{BR} -> Net-(D1-Pad1)
- R13 pad 1: VCC -> GND
- R13 pad 2: /~{BGACK} -> Net-(D2-Pad1)
- R4 pad 2: /68681_Int -> /~{BERR}
- R5 pad 1: Net-(R5-Pad1) -> VCC
- R5 pad 2: Net-(D1-Pad2) -> /~{VPA}
- R6 pad 1: Net-(R6-Pad1) -> VCC
- R6 pad 2: Net-(D5-Pad2) -> /~{HALT}
- R7 pad 1: Net-(R7-Pad1) -> VCC
- R7 pad 2: Net-(D2-Pad2) -> /~{BR}
- R8 pad 1: Net-(R8-Pad1) -> VCC
- R8 pad 2: Net-(D3-Pad2) -> /~{BGACK}
- R9 pad 1: Net-(R9-Pad1) -> VCC
- R9 pad 2: Net-(D4-Pad2) -> /~{DTACK_AVR}
- SW1 pad 2: Net-(C12-Pad1) -> Net-(C1-Pad1)
- U1 pad 10: GND -> unconnected-(U1-Pad10)
- U1 pad 11: unconnected-(U1-Pad11) -> GND
- U1 pad 12: GND -> unconnected-(U1-Pad12)
- U1 pad 2: /~{DS} -> Net-(U1-Pad2)
- U1 pad 3: /~{RAM_WE} -> GND
- U1 pad 4: Net-(U1-Pad4) -> unconnected-(U1-Pad4)
- U1 pad 5: /~{DS} -> GND
- U1 pad 6: /~{OE} -> unconnected-(U1-Pad6)
- U3 pad 1: /A18 -> /A19
- U3 pad 10: GND -> unconnected-(U3-Pad10)
- U3 pad 11: /A17 -> unconnected-(U3-Pad11)
- U3 pad 12: /~{ROMSEL} -> unconnected-(U3-Pad12)
- U3 pad 13: /~{RAMSEL} -> /~{AVRSEL}
- U3 pad 14: /~{UARTSEL} -> /~{RAMSEL}
- U3 pad 15: /~{I2CSEL} -> /~{ROMSEL}
- U3 pad 16: /~{DTACK_CPU} -> VCC
- U3 pad 2: /A19 -> /A20
- U3 pad 3: /A20 -> /A21
- U3 pad 4: /A21 -> GND
- U3 pad 5: /~{AS} -> GND
- U3 pad 6: /~{DTACK_UART} -> VCC
- U3 pad 7: /~{DTACK_I2C} -> unconnected-(U3-Pad7)
- U3 pad 8: /~{DTACK_USER} -> GND
- U3 pad 9: /~{USERSEL} -> unconnected-(U3-Pad9)
- U4 pad 1: /R~{W} -> /~{AVRSEL}
- U4 pad 10: Net-(R5-Pad1) -> GND
- U4 pad 11: /~{I2CSEL} -> GND
- U4 pad 12: Net-(R6-Pad1) -> unconnected-(U4-Pad12)
- U4 pad 13: /~{USERSEL} -> GND
- U4 pad 14: VCC -> GND
- U4 pad 2: Net-(U1-Pad4) -> /~{DTACK_AVR}
- U4 pad 3: /~{ROMSEL} -> /~{AS}
- U4 pad 4: Net-(R7-Pad1) -> /~{DTACK_CPU}
- U4 pad 5: /~{RAMSEL} -> GND
- U4 pad 6: Net-(R8-Pad1) -> GND
- U4 pad 7: GND -> unconnected-(U4-Pad7)
- U4 pad 8: Net-(R9-Pad1) -> GND
- U4 pad 9: /~{UARTSEL} -> unconnected-(U4-Pad9)
- U5 pad 1: unconnected-(U5-Pad1) -> /A18
- U5 pad 10: /~{DTACK_UART} -> /A2
- U5 pad 11: /RxDB -> /A1
- U5 pad 12: unconnected-(U5-Pad12) -> /A0
- U5 pad 13: /TxDB -> /D0
- U5 pad 14: /OP1 -> /D1
- U5 pad 15: /OP3 -> /D2
- U5 pad 16: /OP5 -> GND
- U5 pad 17: /OP7 -> /D3
- U5 pad 18: /D1 -> /D4
- U5 pad 19: /D3 -> /D5
- U5 pad 2: /A0 -> /A16
- U5 pad 20: /D5 -> /D6
- U5 pad 22: GND -> /~{RAMSEL}
- U5 pad 23: unconnected-(U5-Pad23) -> /A10
- U5 pad 24: /68681_Int -> /~{OE}
- U5 pad 25: /D6 -> /A11
- U5 pad 26: /D4 -> /A9
- U5 pad 27: /D2 -> /A8
- U5 pad 28: /D0 -> /A13
- U5 pad 29: /OP6 -> /~{RAM_WE}
- U5 pad 3: /IP3 -> /A14
- U5 pad 30: /OP4 -> /A17
- U5 pad 31: /RTSB -> /A15
- U5 pad 32: /RTSA -> VCC
- U5 pad 4: /A1 -> /A12
- U5 pad 5: /CTSB -> /A7
- U5 pad 6: /A2 -> /A6
- U5 pad 7: /A3 -> /A5
- U5 pad 8: /CTSA -> /A4
- U5 pad 9: /R~{W} -> /A3
- U7 pad 1: /A18 -> /A0
- U7 pad 10: /A2 -> VCC
- U7 pad 11: /A1 -> GND
- U7 pad 12: /A0 -> unconnected-(U7-Pad12)
- U7 pad 13: /D0 -> /CLK
- U7 pad 14: /D1 -> /RXD0
- U7 pad 15: /D2 -> /TXD0
- U7 pad 16: GND -> /R~{W}
- U7 pad 17: /D3 -> /A9
- U7 pad 18: /D4 -> Net-(D2-Pad2)
- U7 pad 19: /D5 -> /IPL0
- U7 pad 2: /A16 -> /A1
- U7 pad 20: /D6 -> /IPL1
- U7 pad 21: /D7 -> /IPL2
- U7 pad 22: /~{RAMSEL} -> /SCL
- U7 pad 23: /A10 -> /SDA
- U7 pad 24: /~{OE} -> /A5
- U7 pad 25: /A11 -> /A6
- U7 pad 26: /A9 -> /A7
- U7 pad 28: /A13 -> /~{DTACK_AVR}
- U7 pad 29: /~{RAM_WE} -> /~{AVRSEL}
- U7 pad 3: /A14 -> /A2
- U7 pad 30: /A17 -> VCC
- U7 pad 31: /A15 -> GND
- U7 pad 32: VCC -> unconnected-(U7-Pad32)
- U7 pad 4: /A12 -> /A3
- U7 pad 5: /A7 -> /A4
- U7 pad 6: /A6 -> /MOSI
- U7 pad 7: /A5 -> /MISO
- U7 pad 8: /A4 -> /SCK
- U7 pad 9: /A3 -> /~{RESET}
- U8 pad 1: Net-(C12-Pad1) -> Net-(C1-Pad1)
- X1 pad 5: /CLK_ONBOARD -> /CLK
Routing:
- net /~{UARTSEL}: track 117.5 -> 0.00 mm, vias 1 -> 0
- net /~{AVRSEL}: track 0.00 -> 116.7 mm
- net /CLK_EXTERNAL: track 116.5 -> 0.00 mm
- net /68681_Int: track 116.0 -> 0.00 mm, vias 2 -> 0
- net /~{VPA}: track 0.00 -> 108.2 mm
- net GND: track 440.8 -> 528.6 mm, vias 21 -> 1
- net /~{OE}: track 84.3 -> 169.5 mm, vias 2 -> 4
- net /~{USERSEL}: track 85.2 -> 0.00 mm
- net /~{DTACK_UART}: track 81.5 -> 0.00 mm, vias 1 -> 0
- net /~{DTACK_USER}: track 64.7 -> 0.00 mm
- net /ERROR: track 63.2 -> 0.00 mm
- net /~{I2CSEL}: track 63.2 -> 0.00 mm, vias 1 -> 0
- net Net-(C13-Pad2): track 62.3 -> 0.00 mm
- net /A5: track 154.2 -> 211.0 mm
- net /A6: track 150.5 -> 207.1 mm
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- removed copper zone on B.Cu, net GND
- removed copper zone on F.Cu, net GND
Other:
- board text added: "MISO"
- board text added: "MOSI"
- board text added: "RX"
- board text added: "SCK"
- board text added: "SCL"
- board text added: "SDA"
- board text added: "TX"
- board text added: "V20220905"
- board text added: "VCC"
- board text added: "~{AVRSEL}"
- board text added: "~{DTACK}"
- board text added: "~{RAMSEL}"
- board text added: "~{RESET}"
- board text added: "~{ROMSEL}"
- board text removed: "CLK Sel"
- board text removed: "ERROR"
- board text removed: "Ex CLK"
- board text removed: "Ext"
- board text removed: "Int"
- board text removed: "V20220621"
- board text removed: "~{DTACK_CPU}"
- board text removed: "~{DTUSER}"
- board text removed: "~{I2CSEL}"
- board text removed: "~{RAM}"
- board text removed: "~{RES}"
- board text removed: "~{ROM}"
- board text removed: "~{UART}"
- board text removed: "~{USEL}"
