File: CPU Board/CPU Board.kicad_pcb (KiCad board)
At the start: 2 copper layers, 99.8 x 99.8 mm, 26 parts, among them J1 Conn_02x32_Odd_Even, U1 GAL16V8, U2 74LS148, U3 GAL16V8, U4 68010D, X1 8Mhz

Commit message: checkpoint
Parts:
- added C10: .1uF, Capacitor_THT:C_Disc_D3.4mm_W2.1mm_P2.50mm, F.Cu at (145.6, 82.0)
- added C11: .1uF, Capacitor_THT:C_Disc_D3.4mm_W2.1mm_P2.50mm, F.Cu at (145.8, 48.8)
- added C7: .1uF, Capacitor_THT:C_Disc_D3.4mm_W2.1mm_P2.50mm, F.Cu at (132.4, 64.3)
- added C8: .1uF, Capacitor_THT:C_Disc_D3.4mm_W2.1mm_P2.50mm, F.Cu at (132.4, 99.6)
- added C9: .1uF, Capacitor_THT:C_Disc_D3.4mm_W2.1mm_P2.50mm, F.Cu at (145.6, 115.6)
- added J2: DEBUG, Connector_PinHeader_2.54mm:PinHeader_1x09_P2.54mm_Vertical, F.Cu at (188.5, 115.6)
- added JP1: DTACK PULLUP, Connector_PinHeader_2.54mm:PinHeader_1x02_P2.54mm_Vertical, F.Cu at (187.7, 63.7)
- added U5: 74LS245, Package_DIP:DIP-20_W7.62mm_Socket_LongPads, F.Cu at (129.8, 68.8)
- added U6: 74LS245, Package_DIP:DIP-20_W7.62mm_Socket_LongPads, F.Cu at (129.8, 104.1)
- added U7: 74LS244, Package_DIP:DIP-20_W7.62mm_Socket_LongPads, F.Cu at (143.0, 120.1)
- added U8: 74LS244, Package_DIP:DIP-20_W7.62mm_Socket_LongPads, F.Cu at (143.0, 86.6)
- added U9: 74LS244, Package_DIP:DIP-20_W7.62mm_Socket_LongPads, F.Cu at (143.0, 53.3)
- moved C4 54.9 mm to (117.3, 115.0)
- moved U3 54.9 mm to (114.8, 119.6)
- moved C3 54.9 mm to (117.3, 81.0)
- moved U1 54.9 mm to (114.8, 85.5)
- moved U2 54.8 mm to (114.8, 57.1)
- moved C2 54.8 mm to (119.9, 52.5)
- moved R5 52.8 mm to (110.2, 55.4)
- moved R6 52.8 mm to (110.2, 74.8)
- moved R7 52.8 mm to (110.2, 86.6)
- moved R2 50.0 mm to (137.4, 58.9), turned to 180 degrees
- moved R9 49.2 mm to (155.7, 127.0), turned to 90 degrees
- moved R3 47.5 mm to (137.4, 54.1), turned to 180 degrees
- moved R10 47.2 mm to (155.7, 116.6), turned to 90 degrees
- moved R8 46.7 mm to (155.7, 106.2), turned to 90 degrees
- moved R11 46.4 mm to (155.7, 95.8), turned to 90 degrees
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Connections:
- J1 pad 54: /D7 -> /BUS_D7
- J1 pad 56: /D6 -> /BUS_D6
- J1 pad 58: /D5 -> /BUS_D5
- J1 pad 60: /D4 -> /BUS_D4
- J1 pad 61: /D0 -> /BUS_D0
- J1 pad 62: /D3 -> /BUS_D3
- J1 pad 63: /D1 -> /BUS_D1
- J1 pad 64: /D2 -> /BUS_D2
- R1 pad 2: VCC -> Net-(R1-Pad2)
Routing:
- net GND: track 0.00 -> 449.0 mm, vias 0 -> 1
- net VCC: track 0.00 -> 440.6 mm
- net /~{AS}: track 0.00 -> 255.0 mm, vias 0 -> 6
- net /D14: track 0.00 -> 249.6 mm, vias 0 -> 4
- net /~{LDS}: track 0.00 -> 231.2 mm, vias 0 -> 1
- net /~{UDS}: track 0.00 -> 225.4 mm, vias 0 -> 4
- net /D12: track 0.00 -> 219.6 mm, vias 0 -> 4
- net /~{HALT}: track 0.00 -> 214.8 mm, vias 0 -> 1
- net /A9: track 0.00 -> 212.6 mm, vias 0 -> 3
- net /R~{W}: track 0.00 -> 202.3 mm, vias 0 -> 3
- net /A13: track 0.00 -> 199.2 mm, vias 0 -> 2
- net /A19: track 0.00 -> 195.7 mm, vias 0 -> 3
- net /CLK: track 0.00 -> 191.7 mm, vias 0 -> 1
- net /A17: track 0.00 -> 180.2 mm, vias 0 -> 5
- net /~{RESET}: track 0.00 -> 178.9 mm, vias 0 -> 1
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Other:
- board text added: "GND"
- board text added: "R~{W}"
- board text added: "V20221107"
- board text added: "~{AS}"
- board text added: "~{BERR}"
- board text added: "~{DTACK}"
- board text added: "~{HALT}"
- board text added: "~{LDS}"
- board text added: "~{RESET}"
- board text added: "~{UDS}"
