File: CPU Board/CPU Board.kicad_pcb (KiCad board)
At the start: 2 copper layers, 99.8 x 99.8 mm, 26 parts, among them J1 Conn_02x32_Odd_Even, U1 GAL16V8, U2 74LS148, U3 GAL16V8, U4 68010D, X1 8Mhz

Commit message: checkpoint
Parts:
- added D1: HALT, LED_THT:LED_D5.0mm, F.Cu at (190.6, 72.0)
- added D2: RUN, LED_THT:LED_D5.0mm, F.Cu at (190.6, 58.0)
- added J2: Conn_01x10, Connector_PinHeader_2.54mm:PinHeader_1x10_P2.54mm_Horizontal, F.Cu at (182.3, 110.7)
- added JP1: DTACK Pullup, Jumper:SolderJumper-2_P1.3mm_Open_RoundedPad1.0x1.5mm, F.Cu at (108.5, 62.7)
- added R12: 470, Resistor_THT:R_Axial_DIN0207_L6.3mm_D2.5mm_P7.62mm_Horizontal, F.Cu at (186.8, 80.1)
- added R13: 470, Resistor_THT:R_Axial_DIN0207_L6.3mm_D2.5mm_P7.62mm_Horizontal, F.Cu at (186.8, 65.8)
- added R4: 4K7, Resistor_THT:R_Axial_DIN0207_L6.3mm_D2.5mm_P7.62mm_Horizontal, F.Cu at (110.2, 93.3)
- moved C4 5.85 mm to (166.4, 114.4)
- moved R2 5.85 mm to (179.1, 75.1)
- moved R3 5.85 mm to (179.1, 55.5)
- moved U2 5.85 mm to (163.8, 56.3)
- moved C2 5.85 mm to (168.8, 51.7)
- moved C3 5.85 mm to (166.4, 80.6)
- moved R5 5.85 mm to (157.0, 51.4)
- moved R6 5.85 mm to (157.0, 70.9)
- moved R7 5.85 mm to (157.0, 82.7)
- moved U1 5.85 mm to (163.8, 85.2)
- moved U3 5.85 mm to (163.8, 119.0)
- moved R9 3.25 mm to (110.2, 112.9)
- moved R10 3.24 mm to (110.2, 109.2)
- moved R8 3.22 mm to (110.2, 100.3)
Connections:
- R1 pad 2: VCC -> Net-(R1-Pad2)
- U3 pad 16: unconnected-(U3-Pad16) -> /~{HALT}
Other:
- board text added: "Debug"
- board text added: "Leaving this un-bridged will allow you to do a freerun test of the cpu board. Once this test passes then bridge this jumper."
- board text added: "Pin 1"
- board text removed: "Steve 68k CPU Board"
