File: CPU Board/CPU Board.kicad_sch (KiCad schematic)
At the start: 26 parts, among them J1 Conn_02x32_Odd_Even, U1 GAL16V8, U2 74LS148, U3 GAL16V8, U4 68010D, X1 8Mhz

Commit message: checkpoint
Parts:
- added C10, C11, C7, C8, C9: .1uF, Capacitor_THT:C_Disc_D3.4mm_W2.1mm_P2.50mm, symbol Device:C
- added J2: DEBUG, Connector_PinHeader_2.54mm:PinHeader_1x09_P2.54mm_Vertical, symbol Connector_Generic:Conn_01x09
- added JP1: DTACK PULLUP, Connector_PinHeader_2.54mm:PinHeader_1x02_P2.54mm_Vertical, symbol Jumper:Jumper_2_Open
- added U5, U6: 74LS245, Package_DIP:DIP-20_W7.62mm_Socket_LongPads, symbol 74xx:74LS245
- added U7, U8, U9: 74LS244, Package_DIP:DIP-20_W7.62mm_Socket_LongPads, symbol 74xx:74LS244
Connections:
- net A1: now also U7.2 (I0a)
- net A10: now also U8.4 (I1a)
- net A11: now also U8.6 (I2a)
- net A12: now also U8.8 (I3a)
- net A13: now also U8.11 (I0b)
- net A14: now also U8.13 (I1b)
- net A15: now also U8.15 (I2b)
- net A16: now also U8.17 (I3b)
- net A17: now also U9.2 (I0a)
- net A18: now also U9.4 (I1a)
- net A19: now also U9.6 (I2a)
- net A2: now also U7.4 (I1a)
- net A20: now also U9.8 (I3a)
- net A21: now also U9.11 (I0b)
- net A22: now also U9.13 (I1b)
- net A23: now also U9.15 (I2b)
- net A3: now also U7.6 (I2a)
- net A4: now also U7.8 (I3a)
- net A5: now also U7.11 (I0b)
- net A6: now also U7.13 (I1b)
- net A7: now also U7.15 (I2b)
- net A8: now also U7.17 (I3b)
- net A9: now also U8.2 (I0a)
- net D0: now also U5.2 (A0); no longer J1.61 (Pin_61)
- net D1: now also U5.3 (A1); no longer J1.63 (Pin_63)
- net D10: now also U6.4 (A2)
- net D11: now also U6.5 (A3)
- net D12: now also U6.6 (A4)
- net D13: now also U6.7 (A5)
- net D14: now also U6.8 (A6)
- net D15: now also U6.9 (A7)
- net D2: now also U5.4 (A2); no longer J1.64 (Pin_64)
- net D3: now also U5.5 (A3); no longer J1.62 (Pin_62)
- net D4: now also U5.6 (A4); no longer J1.60 (Pin_60)
- net D5: now also U5.7 (A5); no longer J1.58 (Pin_58)
- net D6: now also U5.8 (A6); no longer J1.56 (Pin_56)
- net D7: now also U5.9 (A7); no longer J1.54 (Pin_54)
- net D8: now also U6.2 (A0)
- net D9: now also U6.3 (A1)
- net GND: now also C10.2, C11.2, C7.2, C8.2, C9.2, J2.9 (Pin_9), U5.10 (GND), U6.10 (GND), U7.10 (GND), U8.10 (GND), U9.10 (GND), U9.17 (I3b)
- net R~{W}: now also J2.1 (Pin_1), U5.1 (A->B), U6.1 (A->B)
- net VCC: now also C10.1, C11.1, C7.1, C8.1, C9.1, JP1.2 (B), U5.20 (VCC), U6.20 (VCC), U7.20 (VCC), U8.20 (VCC), U9.20 (VCC); no longer R1.2
- net ~{AS}: now also J2.3 (Pin_3), U7.1 (OEa), U7.19 (OEb), U8.1 (OEa), U8.19 (OEb), U9.1 (OEa), U9.19 (OEb)
- net ~{BERR}: now also J2.6 (Pin_6)
- net ~{DTACK}: now also J2.2 (Pin_2)
- net ~{HALT}: now also J2.8 (Pin_8)
- net ~{LDS}: now also J2.5 (Pin_5), U5.19 (CE)
- net ~{RESET}: now also J2.7 (Pin_7)
- net ~{UDS}: now also J2.4 (Pin_4), U6.19 (CE)
- new net: JP1.1 (A), R1.2
- new net BUS_A1: U7.18 (O0a)
- new net BUS_A10: U8.16 (O1a)
- new net BUS_A11: U8.14 (O2a)
- new net BUS_A12: U8.12 (O3a)
- new net BUS_A13: U8.9 (O0b)
- new net BUS_A14: U8.7 (O1b)
- new net BUS_A15: U8.5 (O2b)
- new net BUS_A16: U8.3 (O3b)
- new net BUS_A17: U9.18 (O0a)
- new net BUS_A18: U9.16 (O1a)
- new net BUS_A19: U9.14 (O2a)
- new net BUS_A2: U7.16 (O1a)
- new net BUS_A20: U9.12 (O3a)
- new net BUS_A21: U9.9 (O0b)
- new net BUS_A22: U9.7 (O1b)
- new net BUS_A23: U9.5 (O2b)
- new net BUS_A3: U7.14 (O2a)
- new net BUS_A4: U7.12 (O3a)
- new net BUS_A5: U7.9 (O0b)
- new net BUS_A6: U7.7 (O1b)
- new net BUS_A7: U7.5 (O2b)
- new net BUS_A8: U7.3 (O3b)
- new net BUS_A9: U8.18 (O0a)
- new net BUS_D0: J1.61 (Pin_61), U5.18 (B0)
- new net BUS_D1: J1.63 (Pin_63), U5.17 (B1)
- new net BUS_D10: U6.16 (B2)
- new net BUS_D11: U6.15 (B3)
- new net BUS_D12: U6.14 (B4)
- new net BUS_D13: U6.13 (B5)
- new net BUS_D14: U6.12 (B6)
- new net BUS_D15: U6.11 (B7)
- new net BUS_D2: J1.64 (Pin_64), U5.16 (B2)
- new net BUS_D3: J1.62 (Pin_62), U5.15 (B3)
- new net BUS_D4: J1.60 (Pin_60), U5.14 (B4)
- new net BUS_D5: J1.58 (Pin_58), U5.13 (B5)
- new net BUS_D6: J1.56 (Pin_56), U5.12 (B6)
- new net BUS_D7: J1.54 (Pin_54), U5.11 (B7)
- new net BUS_D8: U6.18 (B0)
- new net BUS_D9: U6.17 (B1)
- no-connect marks 18 -> 19
Other:
- note removed: "Greg@DigicoolThings.com"
- moved on the sheet: C1, C2, C3, C4, C5, C6, H1, H2, H3, H4, R1, R10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
