File: CPU Board/CPU Board.kicad_sch (KiCad schematic)
At the start: 26 parts, among them J1 Conn_02x32_Odd_Even, U1 GAL16V8, U2 74LS148, U3 GAL16V8, U4 68010D, X1 8Mhz

Commit message: More progress
Parts:
- added R?: 4K7, Resistor_THT:R_Axial_DIN0207_L6.3mm_D2.5mm_P7.62mm_Horizontal, symbol Device:R
Connections:
- net VCC: now also R?.1
- net ~{BGACK}: now also R?.2
Changed lines of the file:
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@@
   (junction (at 183.515 23.495) (diameter 0) (color 0 0 0 0)
   )
+  (junction (at 191.135 50.8) (diameter 0) (color 0 0 0 0)
+  )
   (junction (at 62.23 146.685) (diameter 0) (color 0 0 0 0)
   )
@@
   )
   (junction (at 85.09 25.4) (diameter 0) (color 0 0 0 0)
+  )
+  (junction (at 191.135 23.495) (diameter 0) (color 0 0 0 0)
   )
   (junction (at 180.975 119.38) (diameter 0) (color 0 0 0 0)
@@
     (stroke (width 0) (type default) (color 0 0 0 0))
   )
+  (wire (pts (xy 191.135 50.8) (xy 203.2 50.8))
+    (stroke (width 0) (type default) (color 0 0 0 0))
+  )
   (wire (pts (xy 62.23 187.96) (xy 62.23 188.595))
     (stroke (width 0) (type default) (color 0 0 0 0))
@@
     (stroke (width 0) (type default) (color 0 0 0 0))
   )
+  (wire (pts (xy 191.135 23.495) (xy 191.135 28.575))
+    (stroke (width 0) (type default) (color 0 0 0 0))
+  )
   (wire (pts (xy 46.355 159.385) (xy 46.355 179.705))
     (stroke (width 0) (type default) (color 0 0 0 0))
@@
     (stroke (width 0) (type default) (color 0 0 0 0))
   )
+  (wire (pts (xy 188.595 55.88) (xy 203.2 55.88))
+    (stroke (width 0) (type default) (color 0 0 0 0))
+  )
   (wire (pts (xy 229.87 22.86) (xy 229.87 23.495))
     (stroke (width 0) (type default) (color 0 0 0 0))
   )
+  (wire (pts (xy 191.135 36.195) (xy 191.135 50.8))
+    (stroke (width 0) (type default) (color 0 0 0 0))
+  )
   (wire (pts (xy 186.055 81.28) (xy 203.2 81.28))
     (stroke (width 0) (type default) (color 0 0 0 0))
   )
+  (wire (pts (xy 175.895 50.8) (xy 191.135 50.8))
+    (stroke (width 0) (type default) (color 0 0 0 0))
+  )
+  (wire (pts (xy 191.135 23.495) (xy 229.87 23.495))
+    (stroke (width 0) (type default) (color 0 0 0 0))
+  )
   (wire (pts (xy 85.09 24.765) (xy 85.09 25.4))
     (stroke (width 0) (type default) (color 0 0 0 0))
@@
     (stroke (width 0) (type default) (color 0 0 0 0))
   )
-  (wire (pts (xy 203.2 55.88) (xy 188.595 55.88))
-    (stroke (width 0) (type default) (color 0 0 0 0))
-  )
   (wire (pts (xy 31.75 174.625) (xy 43.815 174.625))
     (stroke (width 0) (type default) (color 0 0 0 0))
@@
     (stroke (width 0) (type default) (color 0 0 0 0))
   )
-  (wire (pts (xy 188.595 23.495) (xy 229.87 23.495))
+  (wire (pts (xy 188.595 23.495) (xy 191.135 23.495))
     (stroke (width 0) (type default) (color 0 0 0 0))
   )
@@
     (effects (font (size 1.27 1.27)) (justify left bottom))
   )
+  (label "~{BGACK}" (at 175.895 50.8 180)
+    (effects (font (size 1.27 1.27)) (justify right bottom))
+  )
   (label "~{IRQ4}" (at 36.83 49.53 0)
     (effects (font (size 1.27 1.27)) (justify left bottom))
@@
   )
   (label "~{IRQ2}" (at 31.75 164.465 180)
-    (effects (font (size 1.27 1.27)) (justify right bottom))
-  )
-  (label "~{BGACK}" (at 203.2 50.8 180)
     (effects (font (size 1.27 1.27)) (justify right bottom))
   )
@@
     (pin "1")
   )
+  (symbol (lib_id "Device:R") (at 191.135 32.385 0) (unit 1)
+    (in_bom yes) (on_board yes)
+    (property "Reference" "R?" (id 0) (at 189.865 27.94 90))
+    (property "Value" "4K7" (id 1) (at 191.135 32.385 90)
+      (effects (font (size 1 1)))
+    )
+    (property "Footprint" "Resistor_THT:R_Axial_DIN0207_L6.3mm_D2.5mm_P7.62mm_Horizontal" (id 2) (at 189.357 32.385 90)
+      (effects (font (size 1.27 1.27)) hide)
+    )
+    (property "Datasheet" "~" (id 3) (at 191.135 32.385 0)
+      (effects (font (size 1.27 1.27)) hide)
+    )
+    (pin "1")
+    (pin "2")
+  )
   (symbol (lib_id "power:VCC") (at 75.438 54.991 0) (unit 1)
     (in_bom yes) (on_board yes)
@@
       (reference "R11") (unit 1) (value "4K7") (footprint "Resistor_THT:R_Axial_DIN0207_L6.3mm_D2.5mm_P7.62mm_Horizontal")
     )
+    (path "/66a93d04-0308-433d-84c9-b6bd118d7486"
+      (reference "R?") (unit 1) (value "4K7") (footprint "Resistor_THT:R_Axial_DIN0207_L6.3mm_D2.5mm_P7.62mm_Horizontal")
+    )
     (path "/8495ff12-7ae8-462c-ac90-a118f876eaed"

Commit message: checkpoint
Parts:
- added D1: HALT, LED_THT:LED_D5.0mm, symbol Device:LED
- added D2: RUN, LED_THT:LED_D5.0mm, symbol Device:LED
- added J2: Conn_01x10, Connector_PinHeader_2.54mm:PinHeader_1x10_P2.54mm_Horizontal, symbol Connector_Generic:Conn_01x10
- added JP1: DTACK Pullup, Jumper:SolderJumper-2_P1.3mm_Open_RoundedPad1.0x1.5mm, symbol Jumper:Jumper_2_Open
- added R12, R13: 470, Resistor_THT:R_Axial_DIN0207_L6.3mm_D2.5mm_P7.62mm_Horizontal, symbol Device:R
- gave numbers to parts that had none: 1
Connections:
- net GND: now also J2.1 (Pin_1), J2.10 (Pin_10)
- net R~{W}: now also J2.2 (Pin_2)
- net VCC: now also D1.1 (K), D2.1 (K), JP1.2 (B); no longer R1.2
- net ~{AS}: now also J2.4 (Pin_4)
- net ~{DTACK}: now also J2.3 (Pin_3)
- net ~{HALT}: now also U3.16 (IO4), J2.9 (Pin_9), R12.1
- net ~{IACK}: now also J2.8 (Pin_8)
- net ~{IOSEL}: now also J2.7 (Pin_7)
- net ~{LDS}: now also J2.5 (Pin_5)
- net ~{RUN}: now also R13.1
- net ~{UDS}: now also J2.6 (Pin_6)
- new net: D2.2 (A), R13.2
- new net: JP1.1 (A), R1.2
- new net: D1.2 (A), R12.2
- no-connect marks 18 -> 17
Other:
- note added: "/IACK = /FC0 * /FC1 */FC2 * /A1 * /A2 * A3"
- note added: "/IOSEL = A19 * A20 * A21 * A22 * A23 * /AS /BOOT = GND /RUN = GND"
- note removed: "HALT_STAUTS = /HALT RESET_STATUS = /RESET"
- moved on the sheet: C5, C6, R1

Commit message: V20221121
Parts:
- J2: value Conn_01x10 -> Debug
- R1: value 1k -> 4.7k
Connections:
- net ~{HALT}: no longer U3.16 (IO4)
- no-connect marks 17 -> 18
Other:
- moved on the sheet: D1, D2, R12, R13
