File: IO Board/IO Board.kicad_pcb (KiCad board)
At the start: 2 copper layers, 99.8 x 99.8 mm, 9 parts, among them J1 Conn_02x32_Odd_Even, U1 GAL16V8, U2 68681

Commit message: checkpoint
Parts:
- added C3: 22pf, Capacitor_THT:C_Disc_D3.4mm_W2.1mm_P2.50mm, F.Cu at (139.7, 82.5)
- added C4: 22pf, Capacitor_THT:C_Disc_D3.4mm_W2.1mm_P2.50mm, F.Cu at (139.7, 66.0)
- added J2: DEBUG, Connector_PinHeader_2.54mm:PinHeader_1x09_P2.54mm_Vertical, F.Cu at (159.0, 85.1)
- added J3: UART_A, rosco_m68k:1X06, F.Cu at (158.0, 115.1)
- added J4: UART_B, rosco_m68k:1X06, F.Cu at (158.0, 69.6)
- added Q1: 3.6864MHz, Crystal:Crystal_HC49-4H_Vertical, F.Cu at (141.0, 71.7)
- moved C1 7.61 mm to (123.2, 50.5)
- moved U2 7.61 mm to (116.8, 55.1)
- moved U1 6.87 mm to (120.7, 115.1)
- moved C2 6.86 mm to (123.2, 110.5)
Connections:
- U1 pad 11: /~{DTACKUART} -> unconnected-(U1-Pad11)
- U1 pad 5: /A19 -> /A23
- U1 pad 6: /A20 -> /A22
- U1 pad 8: /A22 -> /A20
- U1 pad 9: /A23 -> /~{DTACKUART}
- U2 pad 10: unconnected-(U2-Pad10) -> /RXDB
- U2 pad 11: unconnected-(U2-Pad11) -> /TXDB
- U2 pad 12: unconnected-(U2-Pad12) -> /RTSB
- U2 pad 13: unconnected-(U2-Pad13) -> /OP3
- U2 pad 14: unconnected-(U2-Pad14) -> /OP5
- U2 pad 15: unconnected-(U2-Pad15) -> /OP7
- U2 pad 2: unconnected-(U2-Pad2) -> /IP3
- U2 pad 26: unconnected-(U2-Pad26) -> /OP6
- U2 pad 27: unconnected-(U2-Pad27) -> /OP4
- U2 pad 28: unconnected-(U2-Pad28) -> /OP2
- U2 pad 29: unconnected-(U2-Pad29) -> /RTSA
- U2 pad 30: unconnected-(U2-Pad30) -> /TXDA
- U2 pad 31: unconnected-(U2-Pad31) -> /RXDA
- U2 pad 32: unconnected-(U2-Pad32) -> Net-(U2-Pad32)
- U2 pad 33: unconnected-(U2-Pad33) -> Net-(U2-Pad33)
- U2 pad 36: unconnected-(U2-Pad36) -> /IP2
- U2 pad 38: unconnected-(U2-Pad38) -> /IP5
- U2 pad 39: unconnected-(U2-Pad39) -> /IP4
- U2 pad 4: unconnected-(U2-Pad4) -> /CTSB
- U2 pad 7: unconnected-(U2-Pad7) -> /CTSA
Routing:
- net GND: track 0.00 -> 220.0 mm
- net VCC: track 0.00 -> 194.1 mm
- net /~{IACK}: track 0.00 -> 174.2 mm
- net /~{DTACKUART}: track 0.00 -> 138.0 mm
- net /A22: track 0.00 -> 125.6 mm
- net /A20: track 0.00 -> 119.0 mm
- net /A23: track 0.00 -> 118.4 mm
- net /A1: track 0.00 -> 115.2 mm
- net /A2: track 0.00 -> 113.6 mm
- net /A21: track 0.00 -> 113.2 mm
- net /A4: track 0.00 -> 112.4 mm
- net /A3: track 0.00 -> 109.2 mm
- net /~{UARTSEL}: track 0.00 -> 103.2 mm
- net /~{IRQ2}: track 0.00 -> 91.7 mm
- net /R~{W}: track 0.00 -> 83.5 mm
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Other:
- board text added: "A20"
- board text added: "A21"
- board text added: "A22"
- board text added: "A23"
- board text added: "GND"
- board text added: "UART A"
- board text added: "UART B"
- board text added: "V20221106"
- board text added: "~{DTACKUART}"
- board text added: "~{IACK}"
- board text added: "~{IRQ2}"
- board text added: "~{UARTSEL}"
