File: IO Board/IO Board.kicad_pcb (KiCad board)
At the start: 2 copper layers, 99.8 x 99.8 mm, 9 parts, among them J1 Conn_02x32_Odd_Even, U1 GAL16V8, U2 68681

Commit message: V20221121
Parts:
- added C3: 15pf, Capacitor_THT:C_Disc_D3.4mm_W2.1mm_P2.50mm, F.Cu at (131.3, 84.1)
- added C4: 5pf, Capacitor_THT:C_Disc_D3.4mm_W2.1mm_P2.50mm, F.Cu at (131.3, 65.3)
- added J2: Serial A, Connector_PinHeader_2.54mm:PinHeader_1x06_P2.54mm_Vertical, F.Cu at (159.5, 119.6)
- added J3: Serial B, Connector_PinHeader_2.54mm:PinHeader_1x06_P2.54mm_Vertical, F.Cu at (146.8, 71.4)
- added J4: DEBUG, Connector_PinHeader_2.54mm:PinHeader_1x09_P2.54mm_Vertical, F.Cu at (170.9, 82.3)
- added J5: Duart IP, Connector_PinHeader_2.54mm:PinHeader_1x08_P2.54mm_Vertical, F.Cu at (132.3, 97.5)
- added J6: Duart OP, Connector_PinHeader_2.54mm:PinHeader_1x06_P2.54mm_Vertical, F.Cu at (132.3, 123.4)
- added Q1: 3.6864MHz, Crystal:Crystal_HC49-4H_Vertical, F.Cu at (132.6, 72.2)
- moved C1 2.79 mm to (112.8, 50.5)
- moved C2 2.79 mm to (113.6, 110.5)
- moved U1 2.79 mm to (111.0, 115.1)
- moved U2 2.79 mm to (106.4, 55.1)
Connections:
- net /~{VPA} renamed /VPA
- J1 pad 12: /~{VMA} -> /~{IOSEL}
- U1 pad 11: /~{DTACKUART} -> unconnected-(U1-Pad11)
- U1 pad 18: /~{DTACK} -> unconnected-(U1-Pad18)
- U1 pad 4: /~{AS} -> /A18
- U1 pad 5: /A19 -> /A17
- U1 pad 6: /A20 -> /A16
- U1 pad 7: /A21 -> /A15
- U1 pad 8: /A22 -> /A14
- U1 pad 9: /A23 -> /~{IOSEL}
- U2 pad 10: unconnected-(U2-Pad10) -> /RXDB
- U2 pad 11: unconnected-(U2-Pad11) -> /TXDB
- U2 pad 12: unconnected-(U2-Pad12) -> /RTSB
- U2 pad 13: unconnected-(U2-Pad13) -> Net-(U2-Pad13)
- U2 pad 14: unconnected-(U2-Pad14) -> Net-(U2-Pad14)
- U2 pad 15: unconnected-(U2-Pad15) -> Net-(U2-Pad15)
- U2 pad 2: unconnected-(U2-Pad2) -> Net-(U2-Pad2)
- U2 pad 26: unconnected-(U2-Pad26) -> Net-(U2-Pad26)
- U2 pad 27: unconnected-(U2-Pad27) -> Net-(U2-Pad27)
- U2 pad 28: unconnected-(U2-Pad28) -> Net-(U2-Pad28)
- U2 pad 29: unconnected-(U2-Pad29) -> /RTSA
- U2 pad 30: unconnected-(U2-Pad30) -> /TXDA
- U2 pad 31: unconnected-(U2-Pad31) -> /RXDA
- U2 pad 32: unconnected-(U2-Pad32) -> Net-(C3-Pad1)
- U2 pad 33: unconnected-(U2-Pad33) -> Net-(C4-Pad1)
- U2 pad 36: unconnected-(U2-Pad36) -> Net-(U2-Pad36)
- U2 pad 38: unconnected-(U2-Pad38) -> Net-(U2-Pad38)
- U2 pad 39: unconnected-(U2-Pad39) -> Net-(U2-Pad39)
- U2 pad 4: unconnected-(U2-Pad4) -> /CTSB
- U2 pad 7: unconnected-(U2-Pad7) -> /CTSA
- U2 pad 9: /~{DTACKUART} -> /~{DTACK}
Routing:
- net GND: track 0.00 -> 234.9 mm, vias 0 -> 1
- net /~{IACK}: track 0.00 -> 173.7 mm
- net VCC: track 0.00 -> 162.6 mm
- net /R~{W}: track 0.00 -> 142.6 mm
- net /~{IOSEL}: track 0.00 -> 130.7 mm
- net /~{LDS}: track 0.00 -> 113.8 mm
- net /~{UARTSEL}: track 0.00 -> 113.7 mm
- net /A1: track 0.00 -> 105.9 mm
- net /A2: track 0.00 -> 104.4 mm
- net /A3: track 0.00 -> 101.8 mm
- net /A4: track 0.00 -> 98.3 mm
- net /~{IRQ2}: track 0.00 -> 96.2 mm
- net /RXDA: track 0.00 -> 94.8 mm
- net /CTSA: track 0.00 -> 91.9 mm, vias 0 -> 1
- net /TXDA: track 0.00 -> 89.9 mm
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Other:
- board text added: "V20221122"
