File: IO Board/IO Board.kicad_sch (KiCad schematic)
At the start: 5 parts, among them J1 Conn_02x32_Odd_Even, U1 GAL16V8, U2 68681

Commit message: checkpoint
Parts:
- added C3, C4: 22pf, Capacitor_THT:C_Disc_D3.4mm_W2.1mm_P2.50mm, symbol Device:C
- added J2: DEBUG, Connector_PinHeader_2.54mm:PinHeader_1x09_P2.54mm_Vertical, symbol Connector_Generic:Conn_01x09
- added J3: UART_A, rosco_m68k:1X06, symbol Connector:Conn_01x06_Male
- added J4: UART_B, rosco_m68k:1X06, symbol Connector:Conn_01x06_Male
- added Q1: 3.6864MHz, Crystal:Crystal_HC49-4H_Vertical, symbol Device:Crystal
Connections:
- net A20: now also J2.5 (Pin_5)
- net A21: now also J2.6 (Pin_6)
- net A22: now also J2.7 (Pin_7)
- net A23: now also J2.8 (Pin_8)
- net GND: now also C3.2, C4.2, J2.9 (Pin_9), J3.1 (Pin_1), J4.1 (Pin_1)
- net VCC: now also J3.3 (Pin_3), J4.3 (Pin_3)
- net ~{DTACKUART}: now also J2.2 (Pin_2)
- net ~{IACK}: now also J2.3 (Pin_3)
- net ~{IRQ2}: now also J2.4 (Pin_4)
- net ~{UARTSEL}: now also J2.1 (Pin_1)
- net RXDB: now reaches U2.10 (RXDB)
- net RXDB: now also J4.4 (Pin_4)
- net TXDB: now reaches U2.11 (TXDB)
- net TXDB: now also J4.5 (Pin_5)
- net RTSB: now reaches U2.12 (OP1)
- net RTSB: now also J4.6 (Pin_6)
- net OP3: now reaches U2.13 (OP3)
- net OP5: now reaches U2.14 (OP5)
- net OP7: now reaches U2.15 (OP7)
- net IP3: now reaches U2.2 (IP3)
- net OP6: now reaches U2.26 (OP6)
- net OP4: now reaches U2.27 (OP4)
- net OP2: now reaches U2.28 (OP2)
- net RTSA: now reaches U2.29 (OP0)
- net RTSA: now also J3.6 (Pin_6)
- net TXDA: now reaches U2.30 (TXDA)
- net TXDA: now also J3.5 (Pin_5)
- net RXDA: now reaches U2.31 (RXDA)
- net RXDA: now also J3.4 (Pin_4)
- net at U2.32 (X1/CLK): now also C3.1, Q1.2
- net at U2.33 (X2): now also C4.1, Q1.1
- net IP2: now reaches U2.36 (IP2)
- net IP5: now reaches U2.38 (IP5)
- net IP4: now reaches U2.39 (IP4)
- net CTSB: now reaches U2.4 (IP1)
- net CTSB: now also J4.2 (Pin_2)
- net CTSA: now reaches U2.7 (IP0)
- net CTSA: now also J3.2 (Pin_2)
Other:
- moved on the sheet: C2
