File: IO Board/IO Board.kicad_sch (KiCad schematic)
At the start: 5 parts, among them J1 Conn_02x32_Odd_Even, U1 GAL16V8, U2 68681

Commit message: checkpoint
Parts:
- added C? (x2): 22pf, symbol Device:C
- added J? (x2): Serial A, symbol Connector_Generic:Conn_01x06
- added J?: DEBUG, symbol Connector_Generic:Conn_01x09
- added Q?: 3.6864MHz, Crystal:Crystal_HC49-4H_Vertical, symbol Device:Crystal
Connections:
- net A20: now also J?.8 (Pin_8)
- net A21: now also J?.7 (Pin_7)
- net A22: now also J?.6 (Pin_6)
- net A23: now also J?.5 (Pin_5)
- net GND: now also C?.2, C?.2, J?.6 (Pin_6), J?.6 (Pin_6), J?.9 (Pin_9)
- net ~{DTACK}: now also U2.9 (DTACK); no longer U1.18 (IO2)
- net ~{IRQ2}: now also J?.2 (Pin_2)
- net ~{UARTSEL}: now also J?.1 (Pin_1)
- net RXDB: now reaches U2.10 (RXDB)
- net RXDB: now also J?.3 (Pin_3)
- net TXDB: now reaches U2.11 (TXDB)
- net TXDB: now also J?.2 (Pin_2)
- net RTSB: now reaches U2.12 (OP1)
- net RTSB: now also J?.5 (Pin_5)
- net RTSA: now reaches U2.29 (OP0)
- net RTSA: now also J?.5 (Pin_5)
- net TXDA: now reaches U2.30 (TXDA)
- net TXDA: now also J?.2 (Pin_2), J?.3 (Pin_3)
- net RXDA: now reaches U2.31 (RXDA)
- net RXDA: now also J?.3 (Pin_3), J?.4 (Pin_4)
- net at U2.32 (X1/CLK): now also C?.1, Q?.2
- net at U2.33 (X2): now also C?.1, Q?.1
- net CTSB: now reaches U2.4 (IP1)
- net CTSB: now also J?.1 (Pin_1)
- net CTSA: now reaches U2.7 (IP0)
- net CTSA: now also J?.1 (Pin_1)
- net ~{DTACKUART}: no longer names the net of U1.9 (I9)
- net ~{DTACKUART}: no longer U2.9 (DTACK)
- no-connect marks 8 -> 11
Other:
- note added: "/UARTSEL = A23 * A22 * A21 * /A20 * /UDS"
- note removed: "/UARTSEL = A23 * A22 * A21 * /A20 * /LDS /DTACK.E = A23 * A22 * A21 * /A20 * /LDS /DTACK.T = /DTACKUART"
- moved on the sheet: C2

Commit message: checkpoint
Parts:
- C3: renamed from C?; value 22pf -> 15pf
- C4: renamed from C?; value 22pf -> 5pf
- gave numbers to parts that had none: 4
Connections:
- net ~{VMA} is gone; now on net ~{IOSEL}: J1.12 (Pin_12)
- net ~{IOSEL}: now reaches U1.9 (I9)
- net ~{VPA renamed VPA
- no-connect marks 11 -> 9
Other:
- moved on the sheet: C1, C2, C3, C4, Q1, U1, U2

Commit message: V20221121
Parts:
- added J5: Duart IP, Connector_PinHeader_2.54mm:PinHeader_1x08_P2.54mm_Vertical, symbol Connector_Generic:Conn_01x06
- added J6: Duart OP, Connector_PinHeader_2.54mm:PinHeader_1x06_P2.54mm_Vertical, symbol Connector_Generic:Conn_01x08
- C3, C4: footprint (none) -> Capacitor_THT:C_Disc_D3.4mm_W2.1mm_P2.50mm
- J2: footprint (none) -> Connector_PinHeader_2.54mm:PinHeader_1x06_P2.54mm_Vertical
- J3: value Serial A -> Serial B; footprint (none) -> Connector_PinHeader_2.54mm:PinHeader_1x06_P2.54mm_Vertical
- J4: footprint (none) -> Connector_PinHeader_2.54mm:PinHeader_1x09_P2.54mm_Vertical
Connections:
- net A14: now also U1.8 (I8)
- net A15: now also U1.7 (I7)
- net A16: now also U1.6 (I6)
- net A17: now also U1.5 (I5)
- net A18: now also U1.4 (I4)
- net A20: no longer J4.8 (Pin_8), U1.8 (I8)
- net A21: no longer J4.7 (Pin_7), U1.7 (I7)
- net A22: no longer J4.6 (Pin_6), U1.6 (I6)
- net A23: no longer J4.5 (Pin_5), U1.5 (I5)
- net GND: now also J5.6 (Pin_6), J6.8 (Pin_8)
- net RXDA: now also J4.5 (Pin_5); no longer J4.4 (Pin_4)
- net R~{W}: now also J4.8 (Pin_8)
- net TXDA: now also J4.4 (Pin_4); no longer J4.3 (Pin_3)
- net VCC: now also J5.1 (Pin_1), J6.1 (Pin_1)
- net ~{AS}: no longer U1.4 (I4)
- net ~{IACK}: now also J4.6 (Pin_6)
- net ~{IOSEL}: now also J4.1 (Pin_1)
- net ~{IRQ2}: now also J4.3 (Pin_3); no longer J4.2 (Pin_2)
- net ~{LDS}: now also J4.7 (Pin_7)
- net ~{UARTSEL}: now also J4.2 (Pin_2); no longer J4.1 (Pin_1)
- net at U2.13 (OP3): now also J6.3 (Pin_3)
- net at U2.14 (OP5): now also J6.5 (Pin_5)
- net at U2.15 (OP7): now also J6.7 (Pin_7)
- net at U2.2 (IP3): now also J5.3 (Pin_3)
- net at U2.26 (OP6): now also J6.6 (Pin_6)
- net at U2.27 (OP4): now also J6.4 (Pin_4)
- net at U2.28 (OP2): now also J6.2 (Pin_2)
- net at U2.36 (IP2): now also J5.2 (Pin_2)
- net at U2.38 (IP5): now also J5.5 (Pin_5)
- net at U2.39 (IP4): now also J5.4 (Pin_4)
Other:
- note added: "/UARTSEL = /IOSEL * /LDS * /A18 * /A17 * /A16 * /A15 * /A14"
- note added: "IO SEL = F80000 (111110000000000000000000) UART = F80001 -"
- note removed: "/UARTSEL = A23 * A22 * A21 * /A20 * /UDS"
- moved on the sheet: J4
