File: RAM and ROM/RAM and ROM.kicad_pcb (KiCad board)
At the start: 2 copper layers, 99.8 x 99.8 mm, 25 parts, among them J1 Conn_02x32_Odd_Even, U1 AS6C4008-55PCN, U2 SST39SF040, U3 GAL16V8, U4 AS6C4008-55PCN, U5 SST39SF040, U6 74HC04

Commit message: checkpoint
Parts:
- added J2: DEBUG, Connector_PinHeader_2.54mm:PinHeader_1x09_P2.54mm_Vertical, F.Cu at (180.3, 54.4)
- D2: value READ -> Read
- D4: value WRITE -> Write
- moved R2 17.5 mm to (172.2, 115.1)
- moved R3 17.5 mm to (172.2, 83.6)
- moved R4 17.5 mm to (172.2, 130.8)
- moved D1 17.5 mm to (180.3, 101.8)
- moved D3 17.5 mm to (180.3, 86.1)
- moved D4 17.5 mm to (180.3, 133.3)
- moved R1 17.5 mm to (172.2, 99.3)
- moved D2 17.5 mm to (180.3, 117.6)
Routing:
- net /A22: track 13.9 -> 132.3 mm, vias 1 -> 0
- net /A23: track 11.4 -> 125.2 mm, vias 0 -> 1
- net /~{ODDROMSEL}: track 77.4 -> 187.7 mm
- net /A20: track 26.4 -> 124.5 mm, vias 0 -> 1
- net /A21: track 21.5 -> 118.7 mm, vias 0 -> 1
- net /D1: track 226.9 -> 151.1 mm, vias 0 -> 1
- net /~{EVENRAMSEL}: track 34.9 -> 96.7 mm
- net Net-(D3-Pad2): track 139.0 -> 83.1 mm, vias 0 -> 1
- net /~{EVENROMSEL}: track 118.5 -> 173.6 mm, vias 0 -> 2
- net /~{ODDRAMSEL}: track 64.0 -> 114.9 mm
- net /R~{W}: track 170.7 -> 215.6 mm
- net Net-(D1-Pad2): track 177.2 -> 134.8 mm, vias 0 -> 1
- net /D7: track 150.9 -> 178.5 mm, vias 1 -> 0
- net /A14: track 167.9 -> 144.4 mm, vias 1 -> 0
- net /A11: track 151.1 -> 174.3 mm, vias 1 -> 0
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Other:
- board text added: "A20"
- board text added: "A21"
- board text added: "A22"
- board text added: "A23"
- board text added: "Address Decode"
- board text added: "Even RAM"
- board text added: "Even ROM"
- board text added: "GND"
- board text added: "Odd RAM"
- board text added: "Odd ROM"
- board text added: "V20221106"
