File: RAM and ROM/RAM and ROM.kicad_pcb (KiCad board)
At the start: 2 copper layers, 99.8 x 99.8 mm, 25 parts, among them J1 Conn_02x32_Odd_Even, U1 AS6C4008-55PCN, U2 SST39SF040, U3 GAL16V8, U4 AS6C4008-55PCN, U5 SST39SF040, U6 74HC04

Commit message: V20221121
Parts:
- removed C5: .1uF, Capacitor_THT:C_Disc_D3.4mm_W2.1mm_P2.50mm
- removed D1: ROMSEL, LED_THT:LED_D5.0mm
- removed D2: READ, LED_THT:LED_D5.0mm
- removed D3: RAMSEL, LED_THT:LED_D5.0mm
- removed D4: WRITE, LED_THT:LED_D5.0mm
- removed R1, R2, R3, R4: 330, Resistor_THT:R_Axial_DIN0207_L6.3mm_D2.5mm_P7.62mm_Horizontal
- removed U6: 74HC04, Package_DIP:DIP-14_W7.62mm_Socket_LongPads
- moved C1 14.0 mm to (168.9, 50.3)
- moved C4 14.0 mm to (168.9, 99.3)
- moved U1 14.0 mm to (162.6, 54.8)
- moved U5 14.0 mm to (162.6, 103.9)
- moved U2 7.64 mm to (133.3, 103.9)
- moved U4 7.64 mm to (133.3, 54.8)
- moved C2 7.64 mm to (139.7, 99.3)
- moved C3 7.64 mm to (139.7, 50.3)
Connections:
- U3 pad 12: /~{RAMSEL} -> unconnected-(U3-Pad12)
- U3 pad 13: /~{ROMSEL} -> unconnected-(U3-Pad13)
Routing:
- net Net-(D1-Pad2): track 177.2 -> 0.00 mm
- net Net-(D3-Pad2): track 139.0 -> 0.00 mm
- net Net-(D4-Pad2): track 103.7 -> 0.00 mm, vias 1 -> 0
- net /R~{W}: track 170.7 -> 76.8 mm
- net /D8: track 109.5 -> 182.1 mm
- net /D1: track 226.9 -> 165.7 mm
- net /D0: track 123.1 -> 174.1 mm, vias 2 -> 0
- net GND: track 365.9 -> 317.3 mm, vias 0 -> 1
- net /D7: track 150.9 -> 194.2 mm, vias 1 -> 0
- net /~{RAMSEL}: track 39.1 -> 0.00 mm
- net /A14: track 167.9 -> 206.1 mm, vias 1 -> 0
- net /~{ROMSEL}: track 35.4 -> 0.00 mm
- net /A9: track 138.4 -> 173.5 mm
- net /D9: track 106.4 -> 137.1 mm, vias 0 -> 1
- net /A18: track 142.5 -> 169.4 mm, vias 1 -> 0
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