File: RAM and ROM/RAM and ROM.kicad_sch (KiCad schematic)
At the start: 25 parts, among them J1 Conn_02x32_Odd_Even, U1 AS6C4008-55PCN, U2 SST39SF040, U3 GAL16V8, U4 AS6C4008-55PCN, U5 SST39SF040, U6 74HC04

Commit message: checkpoint
Parts:
- added J2: DEBUG, Connector_PinHeader_2.54mm:PinHeader_1x09_P2.54mm_Vertical, symbol Connector_Generic:Conn_01x09
Connections:
- net A20: now also J2.5 (Pin_5)
- net A21: now also J2.6 (Pin_6)
- net A22: now also J2.7 (Pin_7)
- net A23: now also J2.8 (Pin_8)
- net GND: now also J2.9 (Pin_9)
- net ~{EVENRAMSEL}: now also J2.3 (Pin_3)
- net ~{EVENROMSEL}: now also J2.1 (Pin_1)
- net ~{ODDRAMSEL}: now also J2.4 (Pin_4)
- net ~{ODDROMSEL}: now also J2.2 (Pin_2)
Changed lines of the file:
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@@
+    (stroke (width 0) (type default) (color 0 0 0 0))
+  )
+  (wire (pts (xy 261.62 151.13) (xy 261.62 154.94))
     (stroke (width 0) (type default) (color 0 0 0 0))
   )
@@
   )
   (wire (pts (xy 165.735 78.105) (xy 165.735 79.375))
+    (stroke (width 0) (type default) (color 0 0 0 0))
+  )
+  (wire (pts (xy 264.795 151.13) (xy 261.62 151.13))
     (stroke (width 0) (type default) (color 0 0 0 0))
   )
@@
     (effects (font (size 1.27 1.27)) (justify left bottom))
   )
+  (label "~{EVENROMSEL}" (at 264.795 130.81 180)
+    (effects (font (size 1.27 1.27)) (justify right bottom))
+  )
   (label "A14" (at 219.075 127.254 180)
     (effects (font (size 1.27 1.27)) (justify right bottom))
@@
     (effects (font (size 1.27 1.27)) (justify left bottom))
   )
+  (label "~{ODDROMSEL}" (at 264.795 133.35 180)
+    (effects (font (size 1.27 1.27)) (justify right bottom))
+  )
   (label "R~{W}" (at 20.701 100.076 180)
     (effects (font (size 1.27 1.27)) (justify right bottom))
@@
     (effects (font (size 1.27 1.27)) (justify right bottom))
   )
+  (label "~{ODDRAMSEL}" (at 264.795 138.43 180)
+    (effects (font (size 1.27 1.27)) (justify right bottom))
+  )
   (label "A12" (at 131.953 122.428 180)
     (effects (font (size 1.27 1.27)) (justify right bottom))
@@
     (effects (font (size 1.27 1.27)) (justify left bottom))
   )
+  (label "A21" (at 264.795 143.51 180)
+    (effects (font (size 1.27 1.27)) (justify right bottom))
+  )
   (label "~{IACK}" (at 43.815 134.62 180)
     (effects (font (size 1.27 1.27)) (justify right bottom))
@@
     (effects (font (size 1.27 1.27)) (justify left bottom))
   )
+  (label "A23" (at 264.795 148.59 180)
+    (effects (font (size 1.27 1.27)) (justify right bottom))
+  )
   (label "D3" (at 113.03 33.655 0)
     (effects (font (size 1.27 1.27)) (justify left bottom))
@@
     (effects (font (size 1.27 1.27)) (justify left bottom))
   )
+  (label "A20" (at 264.795 140.97 180)
+    (effects (font (size 1.27 1.27)) (justify right bottom))
+  )
   (label "A17" (at 131.953 135.128 180)
     (effects (font (size 1.27 1.27)) (justify right bottom))
@@
     (effects (font (size 1.27 1.27)) (justify left bottom))
   )
+  (label "A22" (at 264.795 146.05 180)
+    (effects (font (size 1.27 1.27)) (justify right bottom))
+  )
   (label "A16" (at 87.63 64.135 180)
     (effects (font (size 1.27 1.27)) (justify right bottom))
@@
   (label "D9" (at 249.555 96.774 0)
     (effects (font (size 1.27 1.27)) (justify left bottom))
+  )
+  (label "~{EVENRAMSEL}" (at 264.795 135.89 180)
+    (effects (font (size 1.27 1.27)) (justify right bottom))
   )
   (label "~{WR}" (at 178.435 53.975 0)
@@
     (pin "1")
   )
+  (symbol (lib_id "power:GND") (at 261.62 154.94 0) (unit 1)
+    (in_bom yes) (on_board yes)
+    (property "Reference" "#PWR0115" (id 0) (at 261.62 161.29 0)
+      (effects (font (size 1.27 1.27)) hide)
+    )
+    (property "Value" "GND" (id 1) (at 261.62 158.75 0))
+    (property "Footprint" "" (id 2) (at 261.62 154.94 0)
+      (effects (font (size 1.27 1.27)) hide)
+    )
+    (property "Datasheet" "" (id 3) (at 261.62 154.94 0)
+      (effects (font (size 1.27 1.27)) hide)
+    )
+    (pin "1")
+  )
   (symbol (lib_id "Device:C") (at 192.659 120.396 0) (unit 1)
     (in_bom yes) (on_board yes)
@@
     )
     (pin "1")
+  )
+  (symbol (lib_id "Connector_Generic:Conn_01x09") (at 269.875 140.97 0) (unit 1)
+    (in_bom yes) (on_board yes) (fields_autoplaced)
+    (property "Reference" "J2" (id 0) (at 273.05 139.6999 0)
+      (effects (font (size 1.27 1.27)) (justify left))
+    )
+    (property "Value" "DEBUG" (id 1) (at 273.05 142.2399 0)
+      (effects (font (size 1.27 1.27)) (justify left))
+    )
+    (property "Footprint" "Connector_PinHeader_2.54mm:PinHeader_1x09_P2.54mm_Vertical" (id 2) (at 269.875 140.97 0)
+      (effects (font (size 1.27 1.27)) hide)
+    )
+    (property "Datasheet" "~" (id 3) (at 269.875 140.97 0)
+      (effects (font (size 1.27 1.27)) hide)
+    )
+    (pin "1")
+    (pin "2")
+    (pin "3")
+    (pin "4")
+    (pin "5")
+    (pin "6")
+    (pin "7")
+    (pin "8")
+    (pin "9")
   )
   (symbol (lib_id "power:VCC") (at 147.447 88.646 0) (unit 1)
@@
       (reference "#PWR0114") (unit 1) (value "VCC") (footprint "")
     )
+    (path "/89283502-e13e-4c58-93fe-0e0a0b4dc0b5"
+      (reference "#PWR0115") (unit 1) (value "GND") (footprint "")
+    )
     (path "/cb123b3c-7049-4636-b12e-cfed61d34b5d"
       (reference "C1") (unit 1) (value ".1uF") (footprint "Capacitor_THT:C_Disc_D3.4mm_W2.1mm_P2.50mm")
@@
       (reference "J1") (unit 1) (value "Conn_02x32_Odd_Even") (footprint "Connector_PinHeader_2.54mm:PinHeader_2x32_P2.54mm_Horizontal")
     )
+    (path "/a0407a51-dc9f-4b4e-ba75-441d5c57b182"
+      (reference "J2") (unit 1) (value "DEBUG") (footprint "Connector_PinHeader_2.54mm:PinHeader_1x09_P2.54mm_Vertical")
+    )
     (path "/045f59fc-1a7d-4d13-9615-1bf9766157a2"
