File: RAM and ROM/RAM and ROM.kicad_sch (KiCad schematic)
At the start: 25 parts, among them J1 Conn_02x32_Odd_Even, U1 AS6C4008-55PCN, U2 SST39SF040, U3 GAL16V8, U4 AS6C4008-55PCN, U5 SST39SF040, U6 74HC04

Commit message: V20221121
Parts:
- removed C5: .1uF, Capacitor_THT:C_Disc_D3.4mm_W2.1mm_P2.50mm, symbol Device:C
- removed D1: ROMSEL, LED_THT:LED_D5.0mm, symbol Device:LED
- removed D2, D4: LED, LED_THT:LED_D5.0mm, symbol Device:LED
- removed D3: RAMSEL, LED_THT:LED_D5.0mm, symbol Device:LED
- removed R1, R2, R3, R4: 330, Resistor_THT:R_Axial_DIN0207_L6.3mm_D2.5mm_P7.62mm_Horizontal, symbol Device:R
- removed U6: 74HC04, Package_DIP:DIP-14_W7.62mm_Socket_LongPads, symbol 74xx:74HC04
Connections:
- net ~{RAMSEL}: no longer names the net of U3.12 (IO8)
- net ~{ROMSEL}: no longer names the net of U3.13 (IO7)
- no-connect marks 4 -> 2
Other:
- note added: "/EVENRAM = IACK * /AS * /UDS * /A23 * /A22 * /A21 * /A20 /ODDRAM = IACK * /AS * /LDS * /A23 * /A22 * /A21 * /A20 /EVENROM = IACK * /AS * /UDS * A23 * A22 * A21 * /A20 + IACK * /AS * /UDS /ODDROM = IACK * /AS * /LDS * A23 * A22 * A21 * /A20 + IACK * /AS * /LDS /WR = RW /PPDTACK = IACK * /EVENROM + IACK * /ODDROM + IACK * /EVENRAM + IACK * /ODDRAM DTACK.T = GND DTACK.E = /PPDTACK"
- note removed: "/EVENRAM = IACK * /AS * /UDS * /A23 * /A22 * /A21 * /A20 /ODDRAM = IACK * /AS * /LDS * /A23 * /A22 * /A21 * /A20 /EVENROM = IACK * /AS * /UDS * A23 * A22 * A21 * /A20 + IACK * /AS * /UDS /ODDROM = IACK * /AS * /LDS * A23 * A22 * A21 * /A20 + IACK * /AS * /LDS /WR = RW /PPDTACK = IACK * /EVENROM + IACK * /ODDROM + IACK * /EVENRAM + IACK * /ODDRAM DTACK.T = GND DTACK.E = /PPDTACK /ROMSEL = IACK * /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"
