File: Backplane/Backplane.kicad_pcb (KiCad board)
At the start: 2 copper layers, 99.8 x 99.8 mm, 21 parts, among them J1 Conn_02x32_Odd_Even, J2 Conn_01x06_Male, J3 Conn_02x32_Odd_Even, J4 Conn_02x32_Odd_Even, J5 Conn_02x32_Odd_Even, J6 Conn_02x32_Odd_Even, SW1 Reset, U1 Max705

Commit message: V20221121
Parts:
- added C8: .1uF, Capacitor_THT:C_Disc_D3.4mm_W2.1mm_P2.50mm, F.Cu at (99.6, 73.6)
- added H5: MountingHole, MountingHole:MountingHole_3.2mm_M3, F.Cu at (149.4, 142.6)
- added H6: MountingHole, MountingHole:MountingHole_3.2mm_M3, F.Cu at (149.4, 50.4)
- added X1: 8Mhz, Oscillator:Oscillator_DIP-8, F.Cu at (101.7, 67.0)
- D1: value PWR LED -> Power
- J2: value Conn_01x06_Male -> USB C
- moved SW1 54.8 mm to (108.5, 127.2), turned to 180 degrees
- moved C6 51.8 mm to (112.4, 112.9), turned to -90 degrees
- moved C5 35.9 mm to (109.5, 77.4), turned to 180 degrees
- moved J2 34.7 mm to (107.7, 88.5)
- moved D1 31.1 mm to (103.2, 132.2), turned to -90 degrees
- moved U1 31.0 mm to (101.6, 110.4)
- moved R1 23.0 mm to (110.5, 138.1)
- moved C7 22.4 mm to (98.4, 115.4), turned to 90 degrees
- moved C3 5.84 mm to (166.9, 139.4)
- moved C4 5.84 mm to (183.5, 139.4)
- moved J1 5.84 mm to (189.4, 135.9)
- moved J4 5.84 mm to (176.9, 135.9)
- moved C1 5.84 mm to (126.0, 139.4)
- moved J6 5.84 mm to (115.8, 135.9)
- moved J3 5.84 mm to (156.6, 135.9)
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Connections:
- net /~{VMA} renamed /~{IOSEL}
Routing:
- net GND: track 217.3 -> 0.00 mm
- net VCC: track 152.3 -> 0.00 mm
- net /~{RESET}: track 94.1 -> 0.00 mm
- net /D2: track 91.0 -> 0.00 mm
- net /A3: track 88.6 -> 0.00 mm
- net /CLK: track 79.3 -> 0.00 mm
- net /~{IRQ6}: track 79.3 -> 0.00 mm
- net /~{IRQ5}: track 79.3 -> 0.00 mm
- net /D9: track 79.3 -> 0.00 mm
- net /FC1: track 79.3 -> 0.00 mm
- net /D3: track 79.3 -> 0.00 mm
- net /~{UDS}: track 79.2 -> 0.00 mm
- net /D13: track 79.2 -> 0.00 mm
- net /D15: track 79.2 -> 0.00 mm
- net /~{IRQ4}: track 79.2 -> 0.00 mm
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Other:
- board size 99.8 x 99.8 mm -> 105.9 x 99.8 mm
- board text added: "~{IOSEL}"
- board text removed: "Steve 68k Backplane"
- board text removed: "~{VMA}"
