File: StatusBoard/StatusBoard.kicad_sch (KiCad schematic)
At the start: 45 parts

Commit message: V20221121
Parts:
- removed D?: Read, symbol Device:LED
- removed D?: Write, symbol Device:LED
- removed R? (x2): 470, Resistor_THT:R_Axial_DIN0207_L6.3mm_D2.5mm_P7.62mm_Horizontal, symbol Device:R
- D10, D11, D12, D13, D14, D15, D16, D17, D18, D3, D4, D5, D6, D7, D8, D9: renamed from D?; footprint (none) -> LED_THT:LED_D3.0mm_Clear
- U1, U2, U3: renamed from U?; footprint (none) -> Package_DIP:DIP-20_W7.62mm_Socket_LongPads
- gave numbers to parts that had none: 22
Connections:
- net A14: now also U1.8 (I8)
- net A15: now also U1.7 (I7)
- net A16: now also U1.6 (I6)
- net A17: now also U1.5 (I5)
- net A18: now also U1.4 (I4); no longer U1.9 (I9)
- net A19: no longer U1.8 (I8)
- net A20: no longer U1.7 (I7)
- net A21: no longer U1.6 (I6)
- net A22: no longer U1.5 (I5)
- net A23: no longer U1.4 (I4)
- net ~{IOSEL}: now also U1.9 (I9)
- net ~{VMA}: now reaches J1.8 (Pin_8)
- net ~{STATUSHI} renamed STATUSHI
- net STATUSHI: now also U1.17 (I03); no longer U1.18 (IO2)
- net ~{STATUSLO} renamed STATUSLO
- net STATUSLO: now also U1.18 (IO2); no longer U1.17 (I03)
- no-connect marks 9 -> 10
Other:
- note added: "/STATUSHI = /IOSEL * A18 * /A17 * /A16 * /A15 * /A14 * /UDS /STATUSLO = /IOSEL * A18 * /A17 * /A16 * /A15 * /A14 * /LDS /PPDTACK = /STATUSHI + /STATUSLO DTACK.E = /PPDTACK DTACK.T = GND"
